File: power_suply_shc_1/power_suply_schematic_1.kicad_sch (KiCad schematic)
At the start: 10 parts, among them U1 MCP16301Hx-xCH

Commit message: Add files via upload
Parts:
- C3: value 10 µF -> 10 µF
Connections:
- net +3V3: now also C4.1
- net GND: now also C3.2
Other:
- moved on the sheet: R1, R2

Commit message: Add files via upload
Parts:
- R2: value 33 kΩ -> 31.6 kΩ
Changed lines of the file:
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@@
 			)
 		)
-		(property "Value" "33 kΩ"
+		(property "Value" "31.6 kΩ"
 			(at 176.53 104.1399 0)
 			(effects
