File: rs-232_interface/rs-232_schematic.kicad_sch (KiCad schematic)
At the start: 8 parts, among them J1 6P6C, U1 MAX3232

Commit message: Add files via upload
Parts:
- C1, C2, C3, C4, C5: value C -> 0.1 µF
Connections:
- net GND: now also U1.10 (T2IN), U1.7 (T2OUT), U1.8 (R2IN), U1.9 (R2OUT)
Other:
- moved on the sheet: D1, J1
