File: whole_reader/reader/reader.kicad_sch (KiCad schematic)
At the start: 61 parts, among them U1 LM386, U2 STM32F103C8T6, U3 MCP16301Hx-xCH, U4 MAX3232, Y1 16MHz

Commit message: minor tweaks on board
Parts:
- added SWD1: Conn_01x06_Socket, symbol Connector:Conn_01x06_Socket
Connections:
- net +3.3V: now also SWD1.1 (Pin_1)
- net GND: now also SWD1.6 (Pin_6)
- net RST: now also SWD1.5 (Pin_5)
- net SWCLK: now also SWD1.3 (Pin_3)
- net SWDIO: now also SWD1.2 (Pin_2)
- net TRACESWO: now also SWD1.4 (Pin_4)
Other:
- moved on the sheet: H2
Changed lines of the file:
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@@
 	(symbol
 		(lib_id "Mechanical:MountingHole")
-		(at 100.33 180.34 0)
+		(at 100.33 179.07 0)
 		(unit 1)
 		(exclude_from_sim yes)
@@
 		(fields_autoplaced yes)
 		(property "Reference" "H2"
-			(at 102.87 179.0699 0)
+			(at 102.87 177.7999 0)
 			(effects
 				(font
@@
 		)
 		(property "Value" "MountingHole"
-			(at 102.87 181.6099 0)
+			(at 102.87 180.3399 0)
 			(effects
 				(font
@@
 		)
 		(property "Footprint" "MountingHole:MountingHole_2.2mm_M2"
-			(at 100.33 180.34 0)
+			(at 100.33 179.07 0)
 			(effects
 				(font
@@
 		)
 		(property "Datasheet" "~"
-			(at 100.33 180.34 0)
+			(at 100.33 179.07 0)
 			(effects
 				(font
@@
 		)
 		(property "Description" "Mounting Hole without connection"
-			(at 100.33 180.34 0)
+			(at 100.33 179.07 0)
 			(effects
 				(font
@@
 		(on_board yes)
 		(dnp no)
-		(fields_autoplaced yes)
 		(property "Reference" "#FLG03"
 			(at 78.105 85.09 0)
@@
 		)
 		(property "Value" "PWR_FLAG"
-			(at 76.2 85.0899 90)
+			(at 77.47 81.026 90)
 			(effects
 				(font
@@
 					(unit 1)
 				)
+			)
+		)
+	)
+	(symbol
+		(lib_id "Connector:Conn_01x06_Socket")
+		(at 208.28 101.6 0)
+		(unit 1)
+		(exclude_from_sim no)
+		(in_bom yes)
+		(on_board yes)
+		(dnp no)
+		(fields_autoplaced yes)
+		(property "Reference" "SWD1"
+			(at 209.55 101.5999 0)
+			(effects
+				(font
+					(size 1.27 1.27)
+				)
+				(justify left)
+			)
+		)
+		(property "Value" "Conn_01x06_Socket"
+			(at 209.55 104.1399 0)
+			(effects
+				(font
+					(size 1.27 1.27)
+				)
+				(justify left)
+			)
+		)
+		(property "Footprint" ""
+			(at 208.28 101.6 0)
+			(effects
+				(font
+					(size 1.27 1.27)
+				)
+				(hide yes)
+			)
+		)
+		(property "Datasheet" "~"
+			(at 208.28 101.6 0)
+			(effects
+				(font
+					(size 1.27 1.27)
+				)
+				(hide yes)
+			)
+		)
+		(property "Description" "Generic connector, single row, 01x06, script generated"
+			(at 208.28 101.6 0)
+			(effects
+				(font
+					(size 1.27 1.27)
+				)
+				(hide yes)
+			)
+		)
+		(pin "5"
+		)
+		(pin "2"
+		)
+		(pin "1"
+		)
+		(pin "6"
+		)
+		(pin "3"
+		)
+		(pin "4"
+		)
+		(instances
+			(project ""
+				(path "/6275a1a7-d424-4390-b849-2e49b1a9780b"
+					(reference "SWD1")
+					(unit 1)
+				)

Commit message: Add files via upload
Parts:
- SWD1: value Conn_01x06_Socket -> ~; footprint (none) -> Connector_PinSocket_1.27mm:PinSocket_2x05_P1.27mm_Vertical; symbol Connector:Conn_01x06_Socket -> Connector_Generic:Conn_02x05_Odd_Even
- renumbered SP+1 to +1, SP-1 to -1
Connections:
- net GND: now also SWD1.3 (Pin_3), SWD1.5 (Pin_5), SWD1.9 (Pin_9); no longer SWD1.6 (Pin_6)
- net RST: now also SWD1.10 (Pin_10); no longer SWD1.5 (Pin_5)
- net SWCLK: now also SWD1.4 (Pin_4); no longer SWD1.3 (Pin_3)
- net TRACESWO: now also SWD1.6 (Pin_6); no longer SWD1.4 (Pin_4)
- no-connect marks 26 -> 28
Changed lines of the file:
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@@
 	)
 	(junction
+		(at 199.39 109.22)
+		(diameter 0)
+		(color 0 0 0 0)
+	)
+	(junction
 		(at 229.87 119.38)
 		(diameter 0)
@@
 	)
 	(junction
+		(at 199.39 101.6)
+		(diameter 0)
+		(color 0 0 0 0)
+	)
+	(junction
 		(at 20.32 97.79)
 		(diameter 0)
@@
 	)
 	(no_connect
+		(at 203.2 104.14)
+	)
+	(no_connect
+		(at 215.9 104.14)
+	)
+	(no_connect
 		(at 90.17 130.81)
 	)
@@
 	(wire
 		(pts
+			(xy 203.2 99.06) (xy 199.39 99.06)
+		)
+		(stroke
+			(width 0)
+			(type default)
+		)
+	)
+	(wire
+		(pts
 			(xy 15.24 137.16) (xy 15.24 148.59)
 		)
@@
 	(wire
 		(pts
+			(xy 199.39 109.22) (xy 194.31 109.22)
+		)
+		(stroke
+			(width 0)
+			(type default)
+		)
+	)
+	(wire
+		(pts
 			(xy 128.27 95.25) (xy 128.27 100.33)
 		)
@@
 	(wire
 		(pts
+			(xy 203.2 106.68) (xy 203.2 109.22)
+		)
+		(stroke
+			(width 0)
+			(type default)
+		)
+	)
+	(wire
+		(pts
 			(xy 72.39 184.15) (xy 72.39 185.42)
 		)
@@
 	(wire
 		(pts
-			(xy 203.2 109.22) (xy 194.31 109.22)
+			(xy 203.2 109.22) (xy 199.39 109.22)
 		)
 		(stroke
@@
 	(wire
 		(pts
+			(xy 199.39 99.06) (xy 199.39 101.6)
+		)
+		(stroke
+			(width 0)
+			(type default)
+		)
+	)
+	(wire
+		(pts
 			(xy 33.02 90.17) (xy 40.64 90.17)
 		)
@@
 	(wire
 		(pts
+			(xy 199.39 101.6) (xy 203.2 101.6)
+		)
+		(stroke
+			(width 0)
+			(type default)
+		)
+	)
+	(wire
+		(pts
 			(xy 36.83 115.57) (xy 57.15 115.57)
 		)
@@
 	(wire
 		(pts
+			(xy 199.39 101.6) (xy 199.39 109.22)
+		)
+		(stroke
+			(width 0)
+			(type default)
+		)
+	)
+	(wire
+		(pts
 			(xy 90.17 86.36) (xy 90.17 87.63)
 		)
@@
 	(global_label "TRACESWO"
 		(shape input)
-		(at 203.2 104.14 180)
+		(at 215.9 101.6 0)
 		(fields_autoplaced yes)
 		(effects
@@
 				(size 1.27 1.27)
 			)
-			(justify right)
+			(justify left)
 		)
 		(property "Intersheetrefs" "${INTERSHEET_REFS}"
-			(at 190.4782 104.14 0)
+			(at 228.6218 101.6 0)
 			(effects
 				(font
 					(size 1.27 1.27)
 				)
-				(justify right)
+				(justify left)
 				(hide yes)
 			)
@@
 	(global_label "SWCLK"
 		(shape input)
-		(at 203.2 101.6 180)
+		(at 215.9 99.06 0)
 		(fields_autoplaced yes)
 		(effects
@@
 				(size 1.27 1.27)
 			)
-			(justify right)
+			(justify left)
 		)
 		(property "Intersheetrefs" "${INTERSHEET_REFS}"
-			(at 193.9858 101.6 0)
+			(at 225.1142 99.06 0)
 			(effects
 				(font
 					(size 1.27 1.27)
 				)
-				(justify right)
+				(justify left)
 				(hide yes)
 			)
@@
 	(global_label "SWDIO"
 		(shape input)
-		(at 203.2 99.06 180)
+		(at 215.9 96.52 0)
 		(fields_autoplaced yes)
 		(effects
@@
 				(size 1.27 1.27)
 			)
-			(justify right)
+			(justify left)
 		)
 		(property "Intersheetrefs" "${INTERSHEET_REFS}"
-			(at 194.3486 99.06 0)
+			(at 224.7514 96.52 0)
 			(effects
 				(font
 					(size 1.27 1.27)
 				)
-				(justify right)
+				(justify left)
 				(hide yes)
 			)
@@
 	(global_label "RST"
 		(shape input)
-		(at 203.2 106.68 180)
+		(at 215.9 106.68 0)
 		(fields_autoplaced yes)
 		(effects
@@
 				(size 1.27 1.27)
 			)
-			(justify right)
+			(justify left)
 		)
 		(property "Intersheetrefs" "${INTERSHEET_REFS}"
-			(at 196.7677 106.68 0)
+			(at 222.3323 106.68 0)
 			(effects
 				(font
 					(size 1.27 1.27)
 				)
-				(justify right)
+				(justify left)
 				(hide yes)
 			)
@@
 		(dnp no)
 		(fields_autoplaced yes)
-		(property "Reference" "SP+1"
+		(property "Reference" "+1"
 			(at 85.09 50.1649 90)
 			(effects
@@
 			(project "reader"
 				(path "/6275a1a7-d424-4390-b849-2e49b1a9780b"
-					(reference "SP+1")
+					(reference "+1")
 					(unit 1)
 				)
@@
 		(dnp no)
 		(fields_autoplaced yes)
-		(property "Reference" "SP-1"
+		(property "Reference" "-1"
 			(at 85.09 55.2449 90)
 			(effects
@@
 			(project "reader"
 				(path "/6275a1a7-d424-4390-b849-2e49b1a9780b"
-					(reference "SP-1")
+					(reference "-1")
 					(unit 1)
 				)
@@
 	)
 	(symbol
-		(lib_id "Connector:Conn_01x06_Socket")
+		(lib_id "Connector_Generic:Conn_02x05_Odd_Even")
 		(at 208.28 101.6 0)
 		(unit 1)
@@
 		(fields_autoplaced yes)
 		(property "Reference" "SWD1"
-			(at 209.55 101.5999 0)
+			(at 209.55 92.71 0)
 			(effects
 				(font
 					(size 1.27 1.27)
 				)
-				(justify left)
 			)
 		)
-		(property "Value" "Conn_01x06_Socket"
-			(at 209.55 104.1399 0)
+		(property "Value" "~"
+			(at 209.55 92.71 0)
 			(effects
 				(font
 					(size 1.27 1.27)
 				)
-				(justify left)
 			)
 		)
-		(property "Footprint" ""
+		(property "Footprint" "Connector_PinSocket_1.27mm:PinSocket_2x05_P1.27mm_Vertical"
 			(at 208.28 101.6 0)
 			(effects
@@
 			)
 		)
-		(property "Description" "Generic connector, single row, 01x06, script generated"
+		(property "Description" "Generic connector, double row, 02x05, odd/even pin numbering scheme (row 1 odd numbers, row 2 even numbers), script generated (kicad-library-utils/schlib/autogen/connector/)"
 			(at 208.28 101.6 0)
 			(effects
@@
 		(pin "4"
 		)
+		(pin "9"
+		)
+		(pin "7"
+		)
+		(pin "8"
+		)
+		(pin "10"
+		)
 		(instances
