File: whole_reader/reader/reader.kicad_sch (KiCad schematic)
At the start: 67 parts, among them U1 LM386M-1, U2 STM32F103C8T6, U3 MCP16301Hx-xCH, U4 TP3232N-SR, Y1 16MHz

Commit message: Doplnenie dátových listov a TP sú mimo BOM
Parts:
- C18, C19, C20, C21, C22: value 0.1 µF -> 100 nF; JLCPCB https://jlcpcb.com/partdetail/53938-CL05A105KA5NQNC/C52923 -> https://jlcpcb.com/partdetail/1877-CL05B104KO5NNNC/C1525; LCSC C52923 -> C1525
- RC522: JLCPCB (none) -> https://jlcpcb.com/partdetail/28187-2_54_1_8P/C27438; LCSC (none) -> C27438; now in the parts list
- SWD1: value ~ -> 2x5P, direct insert; JLCPCB (none) -> https://jlcpcb.com/partdetail/Hoauc-2343U205CNG1SNT01/C3502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; LCSC (none) -> C350287
- TP1, TP2, TP3, TP4, TP5: now left out of the parts list
Changed lines of the file:
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@@
 			"AJCGqgIAAAAA2sGpBAAAAADc+qkCAAAAAF1NKQMAAAAA6BgpAwAAAAB0p6sEAAAAACjpugEAAAAA"
 			"ti6sAgAAAABkPkUCAAAAAAD9LAMAAAAAWDtCAgAAAACUMSsDAAAAAMHfrQIAAAAApFWwBAAAAACk"
-			"weEBAAAAAMSmKwMAAAAAti6sAgAAAADwBA=="
+			"weEBAAAAAMSmKwMAAAAAti6sAgAAAADwBAAAAAAAAAAAAAAAAAAAAAAAAAAAAAAAAAAAAAAAAAAA"
+			"AAAAAAAAAAAAAAAAAAAAAAAAAAAAAAAAAAAAAAAAAAAAAAAAAAAAAAAAAAAAAAAAAAAAAAAAAAAA"
+			"AAAAAAAAAAAAAAAAAAAAAAAAAAAAAAAAAAAAAAAAAAAAAAAAAAAAAAAAAAAAAAAAAAAAAAAAAAAA"
+			"AAAAAAAAAAAAAAAAAAAAAAAAAAAAAAAAAAAAAAAAAAAAAAAAAAAAAAAAAAAAAAAAAAAAAAAAAAAA"
+			"AAAAAAAAAAAAAAAAAAAAAAAAAAAAAAAAAAAAAAAAAAAAAAAAAAAAAAAAAAAAAAAAAAAAAAAAAAAA"
+			"AAAAAAAAAAAAAAAAAAAAAAAAAAAAAAAAAAAAAAAAAAAAAAAAAAAAAAAAAAAAAAAAAAAAAAAAAAAA"
+			"AAAAAAAAAAAAAAAAAAAAAAAAAAAAAAAAAAAAAAAAAAAAAAAAAAAAAAAAAAAAAAAAAAAAAAAAAAAA"
+			"AAAAAAAAAAAAAAAAAAAAAAAAAAAAAAAAAAAAAAAAAAAAAAAAAAAAAAAAAAAAAAAAAAAAAAAAAAAA"
+			"AAAAAAAAAAAAAAAAAAAAAAAAAAAAAAAAAAAAAAAAAAAAAAAAAAAAAAAAAAAAAAAAAAAAAAAAAAAA"
+			"AAAAAAAAAAAAAAAAAAAAAAAAAAAAAAAAAAAAAAAAAAAAAAAAAAAAAAAAAAAAAAAAAAAAAAAAAAAA"
+			"AAAAAAAAAAAAAAAAAAAAAAAAAAAAAAAAAAAAAAAAAAAAAAAAAAAAAAAAAAAAAAAAAAAAAAAAAAAA"
+			"AAAAAAAAAAAAAAAAAAAAAAAAAAAAAAAAAAAAAAAAAAAAAAAAAAAAAAAAAAAAAAAAAAAAAAAAAAAA"
+			"AAAAAAAAAAAAAAAAAAAAAAAAAAAAAAAAAAAAAAAAAAAAAAAAAAAAAAAAAAAAAAAAAAAAAAAAAAAA"
+			"AAAAAAAAAAAAAAAAAAAAAAAAAAAAAAAAAAAAAAAAAAAAAAAAAAAAAAAAAAAAAAAAAAAAAAAAAAAA"
+			"AAAAAAAAAAAAAAAAAAAAAAAAAAAAAAAAAAAAAAAAAAAAAAAAAAAAAAAAAAAAAAAAAAAAAAAAAAAA"
+			"AAAAAAAAAAAAAAAAAAAAAAAAAAAAAAAAAAAAAAAAAAAAAAAAAAAAAAAAAAAAAAAAAAAAAAAAAAAA"
+			"AAAAAAAAAAAAAAAAAAAAAAAAAAAAAAAAAAAAAAAAAAAAAAAAAAAAAAAAAAAAAAAAAAAAAAAAAAAA"
+			"AAAAAAAAAAAAAAAAAAAAAAAAAAAAAAAAAAAAAAAAAAAAAAAAAAAAAAAAAAAAAAAAAAAAAAAAAAAA"
+			"AAAAAAAAAAAAAAAAAAAAAAAAAAAAAAAAAA=="
 		)
 	)
@@
 			"AAAAAPRbGECCeuY/iq4UPgAvdX9eXl//c3Nz/wAAAAAAAAAA504GQH8k6T/KBAs+AERqf15eX/9z"
 			"c3P/AAAAAAAAAADmowdAgnrmP4quFD4ALnZ/Xl5f/3Nzc/8AAAAAAAAAAPRbGECCeuY/iq4UPgAv"
-			"dX9eXl//c3Nz/wAAAA=="
+			"dX9eXl//c3Nz/wAAAAAAAAAAAAAAAAAAAAAAAAAAAAAAAAAAAAAAAAAAAAAAAAAAAAAAAAAAAAAA"
+			"AAAAAAAAAAAAAAAAAAAAAAAAAAAAAAAAAAAAAAAAAAAAAAAAAAAAAAAAAAAAAAAAAAAAAAAAAAAA"
+			"AAAAAAAAAAAAAAAAAAAAAAAAAAAAAAAAAAAAAAAAAAAAAAAAAAAAAAAAAAAAAAAAAAAAAAAAAAAA"
+			"AAAAAAAAAAAAAAAAAAAAAAAAAAAAAAAAAAAAAAAAAAAAAAAAAAAAAAAAAAAAAAAAAAAAAAAAAAAA"
+			"AAAAAAAAAAAAAAAAAAAAAAAAAAAAAAAAAAAAAAAAAAAAAAAAAAAAAAAAAAAAAAAAAAAAAAAAAAAA"
+			"AAAAAAAAAAAAAAAAAAAAAAAAAAAAAAAAAAAAAAAAAAAAAAAAAAAAAAAAAAAAAAAAAAAAAAAAAAAA"
+			"AAAAAAAAAAAAAAAAAAAAAAAAAAAAAAAAAAAAAAAAAAAAAAAAAAAAAAAAAAAAAAAAAAAAAAAAAAAA"
+			"AAAAAAAAAAAAAAAAAAAAAAAAAAAAAAAAAAAAAAAAAAAAAAAAAAAAAAAAAAAAAAAAAAAAAAAAAAAA"
+			"AAAAAAAAAAAAAAAAAAAAAAAAAAAAAAAAAAAAAAAAAAAAAAAAAAAAAAAAAAAAAAAAAAAAAAAAAAAA"
+			"AAAAAAAAAAAAAAAAAAAAAAAAAAAAAAAAAAAAAAAAAAAAAAAAAAAAAAAAAAAAAAAAAAAAAAAAAAAA"
+			"AAAAAAAAAAAAAAAAAAAAAAAAAAAAAAAAAAAAAAAAAAAAAAAAAAAAAAAAAAAAAAAAAAAAAAAAAAAA"
+			"AAAAAAAAAAAAAAAAAAAAAAAAAAAAAAAAAAAAAAAAAAAAAAAAAAAAAAAAAAAAAAAAAAAAAAAAAAAA"
+			"AAAAAAAAAAAAAAAAAAAAAAAAAAAAAAAAAAAAAAAAAAAAAAAAAAAAAAAAAAAAAAAAAAAAAAAAAAAA"
+			"AAAAAAAAAAAAAAAAAAAAAAAAAAAAAAAAAAAAAAAAAAAAAAAAAAAAAAAAAAAAAAAAAAAAAAAAAAAA"
+			"AAAAAAAAAAAAAAAAAAAAAAAAAAAAAAAAAAAAAAAAAAAAAAAAAAAAAAAAAAAAAAAAAAAAAAAAAAAA"
+			"AAAAAAAAAAAAAAAAAAAAAAAAAAAAAAAAAAAAAAAAAAAAAAAAAAAAAAAAAAAAAAAAAAAAAAAAAAAA"
+			"AAAAAAAAAAAAAAAAAAAAAAAAAAAAAAAAAAAAAAAAAAAAAAAAAAAAAAAAAAAAAAAAAAAAAAAAAAAA"
+			"AAAAAAAAAAAAAAAAAAAAAAAAAAAAAAAAAAAAAAAAAAAAAAAAAAAAAAAAAAAAAAAAAAAAAAAAAAAA"
+			"AAAAAAAAAAAAAAAAAA=="
 		)
 	)
@@
 			)
 		)
-		(property "Value" "0.1 µF"
+		(property "Value" "100 nF"
 			(at 160.02 39.3699 0)
 			(effects
@@
 			)
 		)
-		(property "Datasheet" "https://jlcpcb.com/api/file/downloadByFileSystemAccessId/8579707174974914560"
+		(property "Datasheet" "https://jlcpcb.com/api/file/downloadByFileSystemAccessId/8579707269996871680"
 			(at 156.21 38.1 0)
 			(effects
@@
 			)
 		)
-		(property "JLCPCB" "https://jlcpcb.com/partdetail/53938-CL05A105KA5NQNC/C52923"
+		(property "JLCPCB" "https://jlcpcb.com/partdetail/1877-CL05B104KO5NNNC/C1525"
 			(at 156.21 38.1 0)
 			(effects
@@
 			)
 		)
-		(property "LCSC" "C52923"
+		(property "LCSC" "C1525"
 			(at 156.21 38.1 0)
 			(effects
@@
 		(unit 1)
 		(exclude_from_sim no)
-		(in_bom yes)
+		(in_bom no)
 		(on_board yes)
 		(dnp no)
@@
 		(unit 1)
 		(exclude_from_sim no)
-		(in_bom no)
+		(in_bom yes)
 		(on_board yes)
 		(dnp no)
@@
 			)
 		)
-		(property "Datasheet" "~"
+		(property "Datasheet" "https://jlcpcb.com/api/file/downloadByFileSystemAccessId/8576018131540119552"
 			(at 269.24 99.06 0)
 			(effects
@@
 			)
 		)
+		(property "JLCPCB" "https://jlcpcb.com/partdetail/28187-2_54_1_8P/C27438"
+			(at 269.24 99.06 0)
+			(effects
+				(font
+					(size 1.27 1.27)
+				)
+			)
+		)
+		(property "LCSC" "C27438"
+			(at 269.24 99.06 0)
+			(effects
+				(font
+					(size 1.27 1.27)
+				)
+			)
+		)
 		(pin "4"
 		)
@@
 			)
 		)
-		(property "Value" "0.1 µF"
+		(property "Value" "100 nF"
 			(at 214.376 40.386 0)
 			(effects
@@
 			)
 		)
-		(property "Datasheet" "https://jlcpcb.com/api/file/downloadByFileSystemAccessId/8579707174974914560"
+		(property "Datasheet" "https://jlcpcb.com/api/file/downloadByFileSystemAccessId/8579707269996871680"
 			(at 212.09 38.1 0)
 			(effects
@@
 			)
 		)
-		(property "JLCPCB" "https://jlcpcb.com/partdetail/53938-CL05A105KA5NQNC/C52923"
+		(property "JLCPCB" "https://jlcpcb.com/partdetail/1877-CL05B104KO5NNNC/C1525"
 			(at 212.09 38.1 0)
 			(effects
@@
 			)
 		)
-		(property "LCSC" "C52923"
+		(property "LCSC" "C1525"
 			(at 212.09 38.1 0)
 			(effects
@@
 		(unit 1)
 		(exclude_from_sim no)
-		(in_bom yes)
+		(in_bom no)
 		(on_board yes)
 		(dnp no)
@@
 		(unit 1)
 		(exclude_from_sim no)
-		(in_bom yes)
+		(in_bom no)
 		(on_board yes)
 		(dnp no)
@@
 		(unit 1)
 		(exclude_from_sim no)
-		(in_bom yes)
+		(in_bom no)
 		(on_board yes)
 		(dnp no)
@@
 			)
 		)
-		(property "Value" "0.1 µF"
+		(property "Value" "100 nF"
 			(at 152.4 30.4799 0)
 			(effects
@@
 			)
 		)
-		(property "Datasheet" "https://jlcpcb.com/api/file/downloadByFileSystemAccessId/8579707174974914560"
+		(property "Datasheet" "https://jlcpcb.com/api/file/downloadByFileSystemAccessId/8579707269996871680"
 			(at 148.59 29.21 0)
 			(effects
@@
 			)
 		)
-		(property "JLCPCB" "https://jlcpcb.com/partdetail/53938-CL05A105KA5NQNC/C52923"
+		(property "JLCPCB" "https://jlcpcb.com/partdetail/1877-CL05B104KO5NNNC/C1525"
 			(at 148.59 29.21 0)
 			(effects
@@
 			)
 		)
-		(property "LCSC" "C52923"
+		(property "LCSC" "C1525"
 			(at 148.59 29.21 0)
 			(effects
@@
 		(unit 1)
 		(exclude_from_sim no)
-		(in_bom yes)
+		(in_bom no)
 		(on_board yes)
 		(dnp no)
@@
 			)
 		)
-		(property "Value" "0.1 µF"
+		(property "Value" "100 nF"
 			(at 216.916 52.324 90)
 			(effects
@@
 			)
 		)
-		(property "Datasheet" "https://jlcpcb.com/api/file/downloadByFileSystemAccessId/8579707174974914560"
+		(property "Datasheet" "https://jlcpcb.com/api/file/downloadByFileSystemAccessId/8579707269996871680"
 			(at 212.09 54.61 0)
 			(effects
@@
 			)
 		)
-		(property "JLCPCB" "https://jlcpcb.com/partdetail/53938-CL05A105KA5NQNC/C52923"
+		(property "JLCPCB" "https://jlcpcb.com/partdetail/1877-CL05B104KO5NNNC/C1525"
 			(at 212.09 54.61 0)
 			(effects
@@
 			)
 		)
-		(property "LCSC" "C52923"
+		(property "LCSC" "C1525"
 			(at 212.09 54.61 0)
 			(effects
@@
 			)
 		)
-		(property "Value" "~"
+		(property "Value" "2x5P, direct insert"
 			(at 209.55 92.71 0)
 			(effects
@@
 			)
 		)
-		(property "Datasheet" "~"
+		(property "Datasheet" "https://jlcpcb.com/api/file/downloadByFileSystemAccessId/8588891463094841344"
 			(at 208.28 101.6 0)
 			(effects
@@
 			)
 		)
+		(property "JLCPCB" "https://jlcpcb.com/partdetail/Hoauc-2343U205CNG1SNT01/C350287"
+			(at 208.28 101.6 0)
+			(effects
+				(font
+					(size 1.27 1.27)
+				)
+			)
+		)
+		(property "LCSC" "C350287"
+			(at 208.28 101.6 0)
+			(effects
+				(font
+					(size 1.27 1.27)
+				)
+			)
+		)
 		(pin "5"
 		)
@@
 			)
 		)
-		(property "Value" "0.1 µF"
+		(property "Value" "100 nF"
 			(at 217.17 44.704 90)
 			(effects
@@
 			)
 		)
-		(property "Datasheet" "https://jlcpcb.com/api/file/downloadByFileSystemAccessId/8579707174974914560"
+		(property "Datasheet" "https://jlcpcb.com/api/file/downloadByFileSystemAccessId/8579707269996871680"
 			(at 212.09 46.99 0)
 			(effects
@@
 			)
 		)
-		(property "JLCPCB" "https://jlcpcb.com/partdetail/53938-CL05A105KA5NQNC/C52923"
+		(property "JLCPCB" "https://jlcpcb.com/partdetail/1877-CL05B104KO5NNNC/C1525"
 			(at 212.09 46.99 0)
 			(effects
@@
 			)
 		)
-		(property "LCSC" "C52923"
+		(property "LCSC" "C1525"
 			(at 212.09 46.99 0)
 			(effects

Commit message: updates on pcb, bom file and experimenting with footprints
Parts:
- BOOT1: JLCPCB https://jlcpcb.com/partdetail/ck-PCM12SMTR/C221841 -> https://jlcpcb.com/partdetail/Alpsalpine-SSSS811101/C109335; LCSC C221841 -> C109335
- L1: JLCPCB https://jlcpcb.com/partdetail/Coilcraft-LPS3010103MRC/C1927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 -> https://jlcpcb.com/partdetail/Ceaiya-CR3012150M/C520285; LCSC C19276043 -> C520285
- LED2: JLCPCB https://jlcpcb.com/partdetail/Kingbright-APHBM2012LSURKZGKC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 -> https://jlcpcb.com/partdetail/Kingbright-APHBM2012SURKCGKC/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; LCSC C6465979 -> C5553822
- R1: JLCPCB https://jlcpcb.com/partdetail/Sunway-SC0805J1003F4ANRH/C315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 -> https://jlcpcb.com/partdetail/160838-0805W8F1003T5E/C149504; LCSC C3152215 -> C149504
- R2: footprint Potentiometer_SMD:Potentiometer_Bourns_3314S_Horizontal -> Potentiometer_SMD:Potentiometer_Bourns_3314G_Vertical
- R3: JLCPCB https://jlcpcb.com/partdetail/25882-0402WGJ0100TCE/C25139 -> https://jlcpcb.com/partdetail/25820-0402WGF100JTCE/C25077; LCSC C25139 -> C25077
- RC522: footprint Connector_PinSocket_2.54mm:PinSocket_1x08_P2.54mm_Vertical -> UACS:PinSocket_1x08_P2.54mm_Vertical
- SWD1: footprint Connector_PinSocket_1.27mm:PinSocket_2x05_P1.27mm_Vertical -> UACS:PinSocket_2x05_P1.27mm_Vertical
- USB-C1: JLCPCB https://jlcpcb.com/partdetail/5762033-USB4110_GFA/C5143397 -> https://jlcpcb.com/partdetail/ShouHan-TYPE_C_16PIN_2MD_073/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; LCSC C5143397 -> C2765186
- Y1: JLCPCB https://jlcpcb.com/partdetail/Yajingxin-TX322516M4DBDE2T/C5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 -> https://jlcpcb.com/partdetail/Yxc_CrystalOscillators-X32251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; LCSC C5310731 -> C13738
Connections:
- net +3.3V: now also SWD1.2 (Pin_2); no longer SWD1.1 (Pin_1)
- net GND: now also SWD1.10 (Pin_10), SWD1.4 (Pin_4), SWD1.6 (Pin_6); no longer SWD1.3 (Pin_3), SWD1.5 (Pin_5), SWD1.9 (Pin_9)
- net NRST: now also SWD1.9 (Pin_9); no longer SWD1.10 (Pin_10)
- net SWCLK: now also SWD1.3 (Pin_3); no longer SWD1.4 (Pin_4)
- net SWDIO: now also SWD1.1 (Pin_1); no longer SWD1.2 (Pin_2)
- net TRACESWO: now also SWD1.5 (Pin_5); no longer SWD1.6 (Pin_6)

Commit message: Úprava popisov
Changed lines of the file:
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@@
 			"MDk0MykoeHkgMy40ODI5MjUgLTMuNTA3NzYxKSh4eSAzLjEzODk2OCAtMi45NTQ1NzgpKHh5IDIu"
 			"OTU3NjY3IC0yLjk0OTIwOSkoeHkgMi43NzYzNjUgLTIuOTQzODQpKHh5IDIuNzc2MzY1IC0zLjc2"
-			"OTkyNikoeHkgLTEuMTQyMjY1IC0zLjc2OQ=="
+			"OTkyNikoeHkgLTEuMTQyMjY1IC0zLjc2OQAAAAAAAAAAAAAAAAAAAAAAAAAAAAAAAAAAAAAAAAAA"
+			"AAAAAAAAAAAAAAAAAAAAAAAAAAAAAAAAAAAAAAAAAAAAAAAAAAAAAAAAAAAAAAAAAAAAAAAAAAAA"
+			"AAAAAAAAAAAAAAAAAAAAAAAAAAAAAAAAAAAAAAAAAAAAAAAAAAAAAAAAAAAAAAAAAAAAAAAAAAAA"
+			"AAAAAAAAAAAAAAAAAAAAAAAAAAAAAAAAAAAAAAAAAAAAAAAAAAAAAAAAAAAAAAAAAAAAAAAAAAAA"
+			"AAAAAAAAAAAAAAAAAAAAAAAAAAAAAAAAAAAAAAAAAAAAAAAAAAAAAAAAAAAAAAAAAAAAAAAAAAAA"
+			"AAAAAAAAAAAAAAAAAAAAAAAAAAAAAAAAAAAAAAAAAAAAAAAAAAAAAAAAAAAAAAAAAAAAAAAAAAAA"
+			"AAAAAAAAAAAAAAAAAAAAAAAAAAAAAAAAAAAAAAAAAAAAAAAAAAAAAAAAAAAAAAAAAAAAAAAAAAAA"
+			"AAAAAAAAAAAAAAAAAAAAAAAAAAAAAAAAAAAAAAAAAAAAAAAAAAAAAAAAAAAAAAAAAAAAAAAAAAAA"
+			"AAAAAAAAAAAAAAAAAAAAAAAAAAAAAAAAAAAAAAAAAAAAAAAAAAAAAAAAAAAAAAAAAAAAAAAAAAAA"
+			"AAAAAAAAAAAAAAAAAAAAAAAAAAAAAAAAAAAAAAAAAAAAAAAAAAAAAAAAAAAAAAAAAAAAAAAAAAAA"
+			"AAAAAAAAAAAAAAAAAAAAAAAAAAAAAAAAAAAAAAAAAAAAAAAAAAAAAAAAAAAAAAAAAAAAAAAAAAAA"
+			"AAAAAAAAAAAAAAAAAAAAAAAAAAAAAAAAAAAAAAAAAAAAAAAAAAAAAAAAAAAAAAAAAAAAAAAAAAAA"
+			"AAAAAAAAAAAAAAAAAAAAAAAAAAAAAAAAAAAAAAAAAAAAAAAAAAAAAAAAAAAAAAAAAAAAAAAAAAAA"
+			"AAAAAAAAAAAAAAAAAAAAAAAAAAAAAAAAAAAAAAAAAAAAAAAAAAAAAAAAAAAAAAAAAAAAAAAAAAAA"
+			"AAAAAAAAAAAAAAAAAAAAAAAAAAAAAAAAAAAAAAAAAAAAAAAAAAAAAAAAAAAAAAAAAAAAAAAAAAAA"
+			"AAAAAAAAAAAAAAAAAAAAAAAAAAAAAAAAAAAAAAAAAAAAAAAAAAAAAAAAAAAAAAAAAAAAAAAAAAAA"
+			"AAAAAAAAAAAAAAAAAAAAAAAAAAAAAAAAAAAAAAAAAAAAAAAAAAAAAAAAAAAAAAAAAAAAAAAAAAAA"
+			"AAAAAAAAAAAAAAAAAAAAAAAAAAAAAAAAAAAAAAAAAAAAAAAAAAAAAAAAAAAAAAAAAAAAAAAAAAAA"
+			"AAAAAAAAAAAAAAAAAAAAAAAAAAAAAAAAAA=="
 		)
 	)
@@
 			"cwBXAEsANwBoAEIAOABwAGcAUAAwAHYAagB1AGgAYQBQADIAMAB2AFQAcwBoAEEAegBkAHAAaQBq"
 			"AHUAaABDAEgAMgAxAGkAagB1AGgAdwBqAGkARgAyAEwAZwBsADMAUQBGAEEAWgB6AEIAQwBSAEwA"
-			"awArADUAdwA0AG8Adw=="
+			"awArADUAdwA0AG8AdwAAAAAAAAAAAAAAAAAAAAAAAAAAAAAAAAAAAAAAAAAAAAAAAAAAAAAAAAAA"
+			"AAAAAAAAAAAAAAAAAAAAAAAAAAAAAAAAAAAAAAAAAAAAAAAAAAAAAAAAAAAAAAAAAAAAAAAAAAAA"
+			"AAAAAAAAAAAAAAAAAAAAAAAAAAAAAAAAAAAAAAAAAAAAAAAAAAAAAAAAAAAAAAAAAAAAAAAAAAAA"
+			"AAAAAAAAAAAAAAAAAAAAAAAAAAAAAAAAAAAAAAAAAAAAAAAAAAAAAAAAAAAAAAAAAAAAAAAAAAAA"
+			"AAAAAAAAAAAAAAAAAAAAAAAAAAAAAAAAAAAAAAAAAAAAAAAAAAAAAAAAAAAAAAAAAAAAAAAAAAAA"
+			"AAAAAAAAAAAAAAAAAAAAAAAAAAAAAAAAAAAAAAAAAAAAAAAAAAAAAAAAAAAAAAAAAAAAAAACAAAA"
+			"AAAAAAAAAAAAAAAAAAAAAAAAAAAAAAAAAAAAAAAAAAAAAAAAAAAAAAAAAAAAAAAAAAAAAAAAAAAA"
+			"AAAAAAAAAAAAAAAAAAAAAAAAAAAAAAAAAAAAAAAAAAAAAAAAAAAAAAAAAAAAAAAAAAAAAAAAAAAA"
+			"AAAAAAAAAAAAAAAAAAAAAAAAAAAAAAAAAAAAAAAAAAAAAAAAAAAAAAAAAAAAAAAAAAAAAAAAAAAA"
+			"AAAAAAAAAAAAAAAAAAAAAAAAAAAAAAAAAAAAAAAAAAAAAAAAAAAAAAAAAAAAAAAAAAAAAAAAAAAA"
+			"AAAAAAAAAAAAAAAAAAAAAAAAAAAAAAAAAAAAAAAAAAAAAAAAAAAAAAAAAAAAAAAAAAAAAAAAAAAA"
+			"AAAAAAAAAAAAAAAAAAAAAAAAAAAAAAAAAAAAAAAAAAAAAAAAAAAAAAAAAAAAAAAAAAAAAAAAAAAA"
+			"AAAAAAAAAAAAAAAAAAAAAAAAAAAAAAAAAAAAAAAAAAAAAAAAAAAAAAAAAAAAAAAAAAAAAAAAAAAA"
+			"AAAAAAAAAAAAAAAAAAAAAAAAAAAAAAAAAAAAAAAAAAAAAAAAAAAAAAAAAAAAAAAAAAAAAAAAAAAA"
+			"AAAAAAAAAAAAAAAAAAAAAAAAAAAAAAAAAAAAAAAAAAAAAAAAAAAAAAAAAAAAAAAAAAAAAAAAAAAA"
+			"AAAAAAAAAAAAAAAAAAAAAAAAAAAAAAAAAAAAAAAAAAAAAAAAAAAAAAAAAAAAAAAAAAAAAAAAAAAA"
+			"AAAAAAAAAAAAAAAAAAAAAAAAAAAAAAAAAAAAAAAAAAAAAAAAAAAAAAAAAAAAAAAAAAAAAAAAAAAA"
+			"AAAAAAAAAAAAAAAAAAAAAAAAAAAAAAAAAAAAAAAAAAAAAAAAAAAAAAAAAAAAAAAAAAAAAAAAAAAA"
+			"AAAAAAAAAAAAAAAAAA=="
 		)
 	)
@@
 		(dnp no)
 		(property "Reference" "SWD1"
-			(at 209.55 92.71 0)
+			(at 209.55 90.424 0)
 			(effects
 				(font
