File: whole_reader/reader/reader.kicad_sch (KiCad schematic)
At the start: 67 parts, among them U1 LM386M-1, U2 STM32F103C8T6, U3 MCP16301Hx-xCH, U4 TP3232N-SR, Y1 16MHz

Commit message: updated values and footprints of rezistors and other parts
Parts:
- C9: footprint Capacitor_SMD:C_0805_2012Metric -> Capacitor_SMD:C_1206_3216Metric; JLCPCB https://jlcpcb.com/partdetail/152991-GRM21BR60J107ME15L/C14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 -> https://jlcpcb.com/partdetail/15681-CL31A107MQHNNNE/C15008; LCSC C141660 -> C15008
- LED2: Note 2mA, Red, Emerald, 120°, SMD-4P, 2 x 1.3 mm -> 20mA, Red, Emerald, 120°, SMD-4P, 2 x 1.3 mm
- R10: JLCPCB https://jlcpcb.com/partdetail/Sunway-SC0603J1002F2BNRH/C315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 -> https://jlcpcb.com/partdetail/26547-0603WAF1002T5E/C25804; LCSC C3152154 -> C25804
- R4: JLCPCB https://jlcpcb.com/partdetail/12862-0402WGJ0331TCE/C12246 -> https://jlcpcb.com/partdetail/25847-0402WGF3300TCE/C25104; LCSC C12246 -> C25104
- R5: value 330 R -> 560 R; footprint Resistor_SMD:R_0402_1005Metric -> Resistor_SMD:R_0603_1608Metric; JLCPCB https://jlcpcb.com/partdetail/12862-0402WGJ0331TCE/C12246 -> https://jlcpcb.com/partdetail/23931-0603WAF5600T5E/C23204; LCSC C12246 -> C23204
- R6: value 330 R -> 56 R; JLCPCB https://jlcpcb.com/partdetail/12862-0402WGJ0331TCE/C12246 -> https://jlcpcb.com/partdetail/25870-0402WGF560JTCE/C25127; LCSC C12246 -> C25127
- R7: value 330 R -> 68 R; JLCPCB https://jlcpcb.com/partdetail/12862-0402WGJ0331TCE/C12246 -> https://jlcpcb.com/partdetail/Yageo-RC0402FR0768RL/C163455; LCSC C12246 -> C163455
- R8: footprint Resistor_SMD:R_0805_2012Metric -> Resistor_SMD:R_0603_1608Metric; JLCPCB https://jlcpcb.com/partdetail/18507-0805W8F7502T5E/C17819 -> https://jlcpcb.com/partdetail/23969-0603WAF7502T5E/C23242; LCSC C17819 -> C23242
- R9: footprint Resistor_SMD:R_0805_2012Metric -> Resistor_SMD:R_0603_1608Metric; JLCPCB https://jlcpcb.com/partdetail/1734-0805W8J0243T5E/C1382 -> https://jlcpcb.com/partdetail/24085-0603WAF2402T5E/C23352; LCSC C1382 -> C23352
Changed lines of the file:
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@@
 			"AAAAAAAAAAAAAAAAAAAAAAAAAAAAAAAAAAAAAAAAAAAAAAAAAAAAAAAAAAAAAAAAAAAAAAAAAAAA"
 			"AAAAAAAAAAAAAAAAAAAAAAAAAAAAAAAAAAAAAAAAAAAAAAAAAAAAAAAAAAAAAAAAAAAAAAAAAAAA"
-			"AAAAAAAAAAAAAAAAAAAAAAAAAAAAAAAAAA=="
+			"AAAAAAAAAAAAAAAAAAAAAAAAAAAAAAAAACzRkgEAAHDuLNGSAQAAwO4s0ZIBAAAQ7yzRkgEAAGDv"
+			"LNGSAQAAsO8s0ZIBAAAA8CzRkgEAAFDwLNGSAQAAoPAs0ZIBAADw8CzRkgEAAPA5Q+2SAQAAMDpD"
+			"7ZIBAABA8SzRkgEAAJDxLNGSAQAAMGcq0ZIBAACwZyrRkgEAAMCVQO2SAQAA4PEs0ZIBAABwTSzR"
+			"kgEAALBNLNGSAQAA8E0s0ZIBAAAwTizRkgEAADDyLNGSAQAAcE4s0ZIBAACwTizRkgEAAPA7Q+2S"
+			"AQAAgPIs0ZIBAADQ8izRkgEAADA8Q+2SAQAAcBFD7ZIBAADwTizRkgEAALA6LNGSAQAAME8s0ZIB"
+			"AABwTyzRkgEAALBPLNGSAQAA8E8s0ZIBAAAwUCzRkgEAACDzLNGSAQAAcPMs0ZIBAADA8yzRkgEA"
+			"ABA7LNGSAQAAcDss0ZIBAADQOyzRkgEAADA8LNGSAQAAEPQs0ZIBAABg9CzRkgEAALD0LNGSAQAA"
+			"APUs0ZIBAABQ9SzRkgEAAKD1LNGSAQAA8PUs0ZIBAABA9izRkgEAAHBQLNGSAQAAsFAs0ZIBAACQ"
+			"PCzRkgEAAPA8LNGSAQAAUD0s0ZIBAACwPSzRkgEAAJD2LNGSAQAA4PYs0ZIBAAAw9yzRkgEAAID3"
+			"LNGSAQAAED4s0ZIBAABwPizRkgEAANA+LNGSAQAAMD8s0ZIBAADQ9yzRkgEAACD4LNGSAQAAcPgs"
+			"0ZIBAADA+CzRkgEAALAfLNGSAQAAkD8s0ZIBAAAwAC3RkgEAAJAALdGSAQAAEPks0ZIBAADwAC3R"
+			"kgEAAFABLdGSAQAAsAEt0ZIBAAAQAi3RkgEAAHACLdGSAQAA0AIt0ZIBAAAwAy3RkgEAAGD5LNGS"
+			"AQAAkAMt0ZIBAADwAy3RkgEAAFAELdGSAQAAsAQt0ZIBAACw+SzRkgEAABAFLdGSAQAAcD5D7ZIB"
+			"AADwUCzRkgEAAPA+Q+2SAQAAMFEs0ZIBAADwTSzRkgEAAAD6LNGSAQAAcAUt0ZIBAABwP0PtkgEA"
+			"ALA/Q+2SAQAAMEBA7ZIBAABwQEDtkgEAAHBRLNGSAQAAsFEs0ZIBAADwUSzRkgEAADBSLNGSAQAA"
+			"sEFA7ZIBAADQBS3RkgEAAICeQO2SAQAAUPos0ZIBAACg+izRkgEAADAGLdGSAQAAkAYt0ZIBAADw"
+			"+izRkgEAADCHLNGSAQAA8EFA7ZIBAADwBi3RkgEAAMA2ItGSAQAAMEJA7ZIBAABwQkDtkgEAAHBS"
+			"LNGSAQAAsFIs0ZIBAABA+yzRkgEAAJD7LNGSAQAAYKBA7ZIBAACwoEDtkgEAAOD7LNGSAQAAMPws"
+			"0ZIBAACA/CzRkgEAAND8LNGSAQAAsIMviw=="
 		)
 	)
@@
 			"AAAAAAAAAAAAAAAAAAAAAAAAAAAAAAAAAAAAAAAAAAAAAAAAAAAAAAAAAAAAAAAAAAAAAAAAAAAA"
 			"AAAAAAAAAAAAAAAAAAAAAAAAAAAAAAAAAAAAAAAAAAAAAAAAAAAAAAAAAAAAAAAAAAAAAAAAAAAA"
+			"AAAAAAAAAAAAAAAAAAAAAAAAAAAAAAAAAAAAAAAAAAAAAAAAAAAAAAAAAAAAAAAAAAAAAAAAAAAA"
+			"AAAAAAAAAAAAAAAAAAAAAAAAAAAAAAAAAAAAAAAAAAAAAAAAAAAAAAAAAAAAAAAAAAAAAAAAAAAA"
+			"AAAAAAAAAAAAAAAAAAAAAAAAAAAAAAAAAAAAAAAAAAAAAAAAAAAAAAAAAAAAAAAAAAAAAAAAAAAA"
+			"AAAAAAAAAAAAAAAAAAAAAAAAAAAAAAAAAAAAAAAAAAAAAAAAAAAAAAAAAAAAAAAAAAAAAAAAAAAA"
+			"AAAAAAAAAAAAAAAAAAAAAAAAAAAAAAAAAAAAAAAAAAAAAAAAAAAAAAAAAAAAAAAAAAAAAAAAAAAA"
+			"AAAAAAAAAAAAAAAAAAAAAAAAAAAAAAAAAAAAAAAAAAAAAAAAAAAAAAAAAAAAAAAAAAAAAAAAAAAA"
+			"AAAAAAAAAAAAAAAAAAAAAAAAAAAAAAAAAAAAAAAAAAAAAAAAAAAAAAAAAAAAAAAAAAAAAAAAAAAA"
+			"AAAAAAAAAAAAAAAAAAAAAAAAAAAAAAAAAAAAAAAAAAAAAAAAAAAAAAAAAAAAAAAAAAAAAAAAAAAA"
+			"AAAAAAAAAAAAAAAAAAAAAAAAAAAAAAAAAAAAAAAAAAAAAAAAAAAAAAAAAAAAAAAAAAAAAAAAAAAA"
+			"AAAAAAAAAAAAAAAAAAAAAAAAAAAAAAAAAAAAAAAAAAAAAAAAAAAAAAAAAAAAAAAAAAAAAAAAAAAA"
+			"AAAAAAAAAAAAAAAAAAAAAAAAAAAAAAAAAAAAAAAAAAAAAAAAAAAAAAAAAAAAAAAAAAAAAAAAAAAA"
+			"AAAAAAAAAAAAAAAAAAAAAAAAAAAAAAAAAAAAAAAAAAAAAAAAAAAAAAAAAAAAAAAAAAAAAAAAAAAA"
+			"AAAAAAAAAAAAAAAAAAAAAAAAAAAAAAAAAAAAAAAAAAAAAAAAAAAAAAAAAAAAAAAAAAAAAAAAAAAA"
+			"AAAAAAAAAAAAAAAAAAAAAAAAAAAAAAAAAAAAAAAAAAAAAAAAAAAAAAAAAAAAAAAAAAAAAAAAAAAA"
+			"AAAAAAAAAAAAAAAAAAAAAAAAAAAAAAAAAAAAAAAAAAAAAAAAAAAAAAAAAAAAAAAAAAAAAAAAAAAA"
+			"AAAAAAAAAAAAAAAAAAAAAAAAAAAAAAAAAAAAAAAAAAAAAAAAAAAAAAAAAAAAAAAAAAAAAAAAAAAA"
+			"AAAAAAAAAAAAAAAAAAAAAAAAAAAAAAAAAAAAAAAAAAAAAAAAAAAAAAAAAAAAAAAAAAAAAAAAAAAA"
+			"AAAAAAAAAAAAAAAAAAAAAAAAAAAAAAAAAAAAAAAAAAAAAAAAAAAAAAAAAAAAAAAAAAAAAAAAAAAA"
 			"AAAAAAAAAAAAAAAAAA=="
 		)
@@
 			)
 		)
-		(property "Datasheet" "https://jlcpcb.com/api/file/downloadByFileSystemAccessId/8588881939923685376"
+		(property "Datasheet" "https://jlcpcb.com/api/file/downloadByFileSystemAccessId/8579706017514917888"
 			(at 105.41 39.37 0)
 			(effects
@@
 			)
 		)
-		(property "JLCPCB" "https://jlcpcb.com/partdetail/12862-0402WGJ0331TCE/C12246"
+		(property "JLCPCB" "https://jlcpcb.com/partdetail/25847-0402WGF3300TCE/C25104"
 			(at 105.41 39.37 0)
 			(effects
@@
 			)
 		)
-		(property "LCSC" "C12246"
+		(property "LCSC" "C25104"
 			(at 105.41 39.37 0)
 			(effects
@@
 			)
 		)
-		(property "Datasheet" "https://jlcpcb.com/api/file/downloadByFileSystemAccessId/8590236309504753664"
+		(property "Datasheet" "https://jlcpcb.com/api/file/downloadByFileSystemAccessId/8579706381320323072"
 			(at 156.21 119.38 0)
 			(effects
@@
 			)
 		)
-		(property "JLCPCB" "https://jlcpcb.com/partdetail/Sunway-SC0603J1002F2BNRH/C3152154"
+		(property "JLCPCB" "https://jlcpcb.com/partdetail/26547-0603WAF1002T5E/C25804"
 			(at 156.21 119.38 0)
 			(effects
@@
 			)
 		)
-		(property "LCSC" "C3152154"
+		(property "LCSC" "C25804"
 			(at 156.21 119.38 0)
 			(effects
@@
 			)
 		)
-		(property "Footprint" "Capacitor_SMD:C_0805_2012Metric"
+		(property "Footprint" "Capacitor_SMD:C_1206_3216Metric"
 			(at 78.74 46.0248 0)
 			(effects
@@
 			)
 		)
-		(property "Datasheet" "https://jlcpcb.com/api/file/downloadByFileSystemAccessId/8588894212876484608"
+		(property "Datasheet" "https://jlcpcb.com/api/file/downloadByFileSystemAccessId/8586178582331215872"
 			(at 74.93 46.99 0)
 			(effects
@@
 			)
 		)
-		(property "JLCPCB" "https://jlcpcb.com/partdetail/152991-GRM21BR60J107ME15L/C141660"
+		(property "JLCPCB" "https://jlcpcb.com/partdetail/15681-CL31A107MQHNNNE/C15008"
 			(at 74.93 46.99 0)
 			(effects
@@
 			)
 		)
-		(property "LCSC" "C141660"
+		(property "LCSC" "C15008"
 			(at 74.93 46.99 0)
 			(effects
@@
 			)
 		)
-		(property "Footprint" "Resistor_SMD:R_0805_2012Metric"
+		(property "Footprint" "Resistor_SMD:R_0603_1608Metric"
 			(at 167.132 168.91 90)
 			(effects
@@
 			)
 		)
-		(property "Datasheet" "https://jlcpcb.com/api/file/downloadByFileSystemAccessId/8579706657955778560"
+		(property "Datasheet" "https://jlcpcb.com/api/file/downloadByFileSystemAccessId/8579706316903792640"
 			(at 168.91 168.91 0)
 			(effects
@@
 			)
 		)
-		(property "JLCPCB" "https://jlcpcb.com/partdetail/18507-0805W8F7502T5E/C17819"
+		(property "JLCPCB" "https://jlcpcb.com/partdetail/23969-0603WAF7502T5E/C23242"
 			(at 168.91 168.91 0)
 			(effects
@@
 			)
 		)
-		(property "LCSC" " C17819"
+		(property "LCSC" "C23242"
 			(at 168.91 168.91 0)
 			(effects
@@
 			)
 		)
-		(property "Value" "330 R"
+		(property "Value" "56 R"
 			(at 125.476 37.592 90)
 			(effects
@@
 			)
 		)
-		(property "Datasheet" "https://jlcpcb.com/api/file/downloadByFileSystemAccessId/8588881939923685376"
+		(property "Datasheet" "https://jlcpcb.com/api/file/downloadByFileSystemAccessId/8586178279397068800"
 			(at 128.27 39.37 0)
 			(effects
@@
 			)
 		)
-		(property "JLCPCB" "https://jlcpcb.com/partdetail/12862-0402WGJ0331TCE/C12246"
+		(property "JLCPCB" "https://jlcpcb.com/partdetail/25870-0402WGF560JTCE/C25127"
 			(at 128.27 39.37 0)
 			(effects
@@
 			)
 		)
-		(property "LCSC" "C12246"
+		(property "LCSC" "C25127"
 			(at 128.27 39.37 0)
 			(effects
@@
 			)
 		)
-		(property "Note" "2mA, Red, Emerald, 120°, SMD-4P, 2 x 1.3 mm"
+		(property "Note" "20mA, Red, Emerald, 120°, SMD-4P, 2 x 1.3 mm"
 			(at 130.81 54.61 0)
 			(effects
@@
 			)
 		)
-		(property "Value" "330 R"
+		(property "Value" "68 R"
 			(at 136.398 37.846 90)
 			(effects
@@
 			)
 		)
-		(property "Datasheet" "https://jlcpcb.com/api/file/downloadByFileSystemAccessId/8588881939923685376"
+		(property "Datasheet" "https://jlcpcb.com/api/file/downloadByFileSystemAccessId/8588908782960693248"
 			(at 133.35 39.37 0)
 			(effects
@@
 			)
 		)
-		(property "JLCPCB" "https://jlcpcb.com/partdetail/12862-0402WGJ0331TCE/C12246"
+		(property "JLCPCB" "https://jlcpcb.com/partdetail/Yageo-RC0402FR0768RL/C163455"
 			(at 133.35 39.37 0)
 			(effects
@@
 			)
 		)
-		(property "LCSC" "C12246"
+		(property "LCSC" "C163455"
 			(at 133.35 39.37 0)
 			(effects
@@
 			)
 		)
-		(property "Footprint" "Resistor_SMD:R_0805_2012Metric"
+		(property "Footprint" "Resistor_SMD:R_0603_1608Metric"
 			(at 167.132 182.88 90)
 			(effects
@@
 			)
 		)
-		(property "Datasheet" "https://jlcpcb.com/api/file/downloadByFileSystemAccessId/8588881938798530560"
+		(property "Datasheet" "https://jlcpcb.com/api/file/downloadByFileSystemAccessId/8579706339318288384"
 			(at 168.91 182.88 0)
 			(effects
@@
 			)
 		)
-		(property "JLCPCB" "https://jlcpcb.com/partdetail/1734-0805W8J0243T5E/C1382"
+		(property "JLCPCB" "https://jlcpcb.com/partdetail/24085-0603WAF2402T5E/C23352"
 			(at 168.91 182.88 0)
 			(effects
@@
 			)
 		)
-		(property "LCSC" "C1382"
+		(property "LCSC" "C23352"
 			(at 168.91 182.88 0)
 			(effects
@@
 			)
 		)
-		(property "Value" "330 R"
+		(property "Value" "560 R"
 			(at 113.03 37.846 90)
 			(effects
@@
 			)
 		)
-		(property "Footprint" "Resistor_SMD:R_0402_1005Metric"
+		(property "Footprint" "Resistor_SMD:R_0603_1608Metric"
 			(at 108.712 39.37 90)
 			(effects
@@
 			)
 		)
-		(property "Datasheet" "https://jlcpcb.com/api/file/downloadByFileSystemAccessId/8588881939923685376"
+		(property "Datasheet" "https://jlcpcb.com/api/file/downloadByFileSystemAccessId/8579706294262939648"
 			(at 110.49 39.37 0)
 			(effects
@@
 			)
 		)
-		(property "JLCPCB" "https://jlcpcb.com/partdetail/12862-0402WGJ0331TCE/C12246"
+		(property "JLCPCB" "https://jlcpcb.com/partdetail/23931-0603WAF5600T5E/C23204"
 			(at 110.49 39.37 0)
 			(effects
@@
 			)
 		)
-		(property "LCSC" "C12246"
+		(property "LCSC" "C23204"
 			(at 110.49 39.37 0)
 			(effects

Commit message: added speaker to the schematics
Parts:
- added LS1: Speaker, symbol Device:Speaker
Changed lines of the file:
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@@
 			"+izRkgEAADCHLNGSAQAA8EFA7ZIBAADwBi3RkgEAAMA2ItGSAQAAMEJA7ZIBAABwQkDtkgEAAHBS"
 			"LNGSAQAAsFIs0ZIBAABA+yzRkgEAAJD7LNGSAQAAYKBA7ZIBAACwoEDtkgEAAOD7LNGSAQAAMPws"
-			"0ZIBAACA/CzRkgEAAND8LNGSAQAAsIMviw=="
+			"0ZIBAACA/CzRkgEAAND8LNGSAQAAsIMviwAAAAAAAAAAAAAAAAAAAAAAAAAAAAAAAAAAAAAAAAAA"
+			"AAAAAAAAAAAAAAAAAAAAAAAAAAAAAAAAAAAAAAAAAAAAAAAAAAAAAAAAAAAAAAAAAAAAAAAAAAAA"
+			"AAAAAAAAAAAAAAAAAAAAAAAAAAAAAAAAAAAAAAAAAAAAAAAAAAAAAAAAAAAAAAAAAAAAAAAAAAAA"
+			"AAAAAAAAAAAAAAAAAAAAAAAAAAAAAAAAAAAAAAAAAAAAAAAAAAAAAAAAAAAAAAAAAAAAAAAAAAAA"
+			"AAAAAAAAAAAAAAAAAAAAAAAAAAAAAAAAAAAAAAAAAAAAAAAAAAAAAAAAAAAAAAAAAAAAAAAAAAAA"
+			"AAAAAAAAAAAAAAAAAAAAAAAAAAAAAAAAAAAAAAAAAAAAAAAAAAAAAAAAAAAAAAAAAAAAAAAAAAAA"
+			"AAAAAAAAAAAAAAAAAAAAAAAAAAAAAAAAAAAAAAAAAAAAAAAAAAAAAAAAAAAAAAAAAAAAAAAAAAAA"
+			"AAAAAAAAAAAAAAAAAAAAAAAAAAAAAAAAAAAAAAAAAAAAAAAAAAAAAAAAAAAAAAAAAAAAAAAAAAAA"
+			"AAAAAAAAAAAAAAAAAAAAAAAAAAAAAAAAAAAAAAAAAAAAAAAAAAAAAAAAAAAAAAAAAAAAAAAAAAAA"
+			"AAAAAAAAAAAAAAAAAAAAAAAAAAAAAAAAAAAAAAAAAAAAAAAAAAAAAAAAAAAAAAAAAAAAAAAAAAAA"
+			"AAAAAAAAAAAAAAAAAAAAAAAAAAAAAAAAAAAAAAAAAAAAAAAAAAAAAAAAAAAAAAAAAAAAAAAAAAAA"
+			"AAAAAAAAAAAAAAAAAAAAAAAAAAAAAAAAAAAAAAAAAAAAAAAAAAAAAAAAAAAAAAAAAAAAAAAAAAAA"
+			"AAAAAAAAAAAAAAAAAAAAAAAAAAAAAAAAAAAAAAAAAAAAAAAAAAAAAAAAAAAAAAAAAAAAAAAAAAAA"
+			"AAAAAAAAAAAAAAAAAAAAAAAAAAAAAAAAAAAAAAAAAAAAAAAAAAAAAAAAAAAAAAAAAAAAAAAAAAAA"
+			"AAAAAAAAAAAAAAAAAAAAAAAAAAAAAAAAAAAAAAAAAAAAAAAAAAAAAAAAAAAAAAAAAAAAAAAAAAAA"
+			"AAAAAAAAAAAAAAAAAAAAAAAAAAAAAAAAAAAAAAAAAAAAAAAAAAAAAAAAAAAAAAAAAAAAAAAAAAAA"
+			"AAAAAAAAAAAAAAAAAAAAAAAAAAAAAAAAAAAAAAAAAAAAAAAAAAAAAAAAAAAAAAAAAAAAAAAAAAAA"
+			"AAAAAAAAAAAAAAAAAAAAAAAAAAAAAAAAAAAAAAAAAAAAAAAAAAAAAAAAAAAAAAAAAAAAAAAAAAAA"
+			"AAAAAAAAAAAAAAAAAAAAAAAAAAAAAAAAAA=="
 		)
 	)
@@
 			"AAAAAAAAAAAAAAAAAAAAAAAAAAAAAAAAAAAAAAAAAAAAAAAAAAAAAAAAAAAAAAAAAAAAAAAAAAAA"
 			"AAAAAAAAAAAAAAAAAAAAAAAAAAAAAAAAAAAAAAAAAAAAAAAAAAAAAAAAAAAAAAAAAAAAAAAAAAAA"
+			"AAAAAAAAAAAAAAAAAAAAAAAAAAAAAAAAAAAAAAAAAAAAAAAAAAAAAAAAAAAAAAAAAAAAAAAAAAAA"
+			"AAAAAAAAAAAAAAAAAAAAAAAAAAAAAAAAAAAAAAAAAAAAAAAAAAAAAAAAAAAAAAAAAAAAAAAAAAAA"
+			"AAAAAAAAAAAAAAAAAAAAAAAAAAAAAAAAAAAAAAAAAAAAAAAAAAAAAAAAAAAAAAAAAAAAAAAAAAAA"
+			"AAAAAAAAAAAAAAAAAAAAAAAAAAAAAAAAAAAAAAAAAAAAAAAAAAAAAAAAAAAAAAAAAAAAAAAAAAAA"
+			"AAAAAAAAAAAAAAAAAAAAAAAAAAAAAAAAAAAAAAAAAAAAAAAAAAAAAAAAAAAAAAAAAAAAAAAAAAAA"
+			"AAAAAAAAAAAAAAAAAAAAAAAAAAAAAAAAAAAAAAAAAAAAAAAAAAAAAAAAAAAAAAAAAAAAAAAAAAAA"
+			"AAAAAAAAAAAAAAAAAAAAAAAAAAAAAAAAAAAAAAAAAAAAAAAAAAAAAAAAAAAAAAAAAAAAAAAAAAAA"
+			"AAAAAAAAAAAAAAAAAAAAAAAAAAAAAAAAAAAAAAAAAAAAAAAAAAAAAAAAAAAAAAAAAAAAAAAAAAAA"
+			"AAAAAAAAAAAAAAAAAAAAAAAAAAAAAAAAAAAAAAAAAAAAAAAAAAAAAAAAAAAAAAAAAAAAAAAAAAAA"
+			"AAAAAAAAAAAAAAAAAAAAAAAAAAAAAAAAAAAAAAAAAAAAAAAAAAAAAAAAAAAAAAAAAAAAAAAAAAAA"
+			"AAAAAAAAAAAAAAAAAAAAAAAAAAAAAAAAAAAAAAAAAAAAAAAAAAAAAAAAAAAAAAAAAAAAAAAAAAAA"
+			"AAAAAAAAAAAAAAAAAAAAAAAAAAAAAAAAAAAAAAAAAAAAAAAAAAAAAAAAAAAAAAAAAAAAAAAAAAAA"
+			"AAAAAAAAAAAAAAAAAAAAAAAAAAAAAAAAAAAAAAAAAAAAAAAAAAAAAAAAAAAAAAAAAAAAAAAAAAAA"
+			"AAAAAAAAAAAAAAAAAAAAAAAAAAAAAAAAAAAAAAAAAAAAAAAAAAAAAAAAAAAAAAAAAAAAAAAAAAAA"
+			"AAAAAAAAAAAAAAAAAAAAAAAAAAAAAAAAAAAAAAAAAAAAAAAAAAAAAAAAAAAAAAAAAAAAAAAAAAAA"
+			"AAAAAAAAAAAAAAAAAAAAAAAAAAAAAAAAAAAAAAAAAAAAAAAAAAAAAAAAAAAAAAAAAAAAAAAAAAAA"
+			"AAAAAAAAAAAAAAAAAAAAAAAAAAAAAAAAAAAAAAAAAAAAAAAAAAAAAAAAAAAAAAAAAAAAAAAAAAAA"
+			"AAAAAAAAAAAAAAAAAAAAAAAAAAAAAAAAAAAAAAAAAAAAAAAAAAAAAAAAAAAAAAAAAAAAAAAAAAAA"
 			"AAAAAAAAAAAAAAAAAA=="
 		)
@@
 	)
 	(symbol
+		(lib_id "Device:Speaker")
+		(at 86.36 54.61 0)
+		(unit 1)
+		(exclude_from_sim no)
+		(in_bom yes)
+		(on_board no)
+		(dnp yes)
+		(fields_autoplaced yes)
+		(property "Reference" "LS1"
+			(at 91.44 54.6099 0)
+			(effects
+				(font
+					(size 1.27 1.27)
+				)
+				(justify left)
+			)
+		)
+		(property "Value" "Speaker"
+			(at 91.44 57.1499 0)
+			(effects
+				(font
+					(size 1.27 1.27)
+				)
+				(justify left)
+			)
+		)
+		(property "Footprint" ""
+			(at 86.36 59.69 0)
+			(effects
+				(font
+					(size 1.27 1.27)
+				)
+				(hide yes)
+			)
+		)
+		(property "Datasheet" "https://jlcpcb.com/api/file/downloadByFileSystemAccessId/8600630112542994432"
+			(at 86.106 55.88 0)
+			(effects
+				(font
+					(size 1.27 1.27)
+				)
+				(hide yes)
+			)
+		)
+		(property "Description" "Speaker"
+			(at 86.36 54.61 0)
+			(effects
+				(font
+					(size 1.27 1.27)
+				)
+				(hide yes)
+			)
+		)
+		(property "Field5" ""
+			(at 86.36 54.61 0)
+			(effects
+				(font
+					(size 1.27 1.27)
+				)
+				(hide yes)
+			)
+		)
+		(property "Field6" ""
+			(at 86.36 54.61 0)
+			(effects
+				(font
+					(size 1.27 1.27)
+				)
+				(hide yes)
+			)
+		)
+		(property "JLCPCB" "https://jlcpcb.com/partdetail/Dragonstate-HDK_100832011/C19725762"
+			(at 86.36 54.61 0)
+			(effects
+				(font
+					(size 1.27 1.27)
+				)
+				(hide yes)
+			)
+		)
+		(property "LCSC" "C19725762"
+			(at 86.36 54.61 0)
+			(effects
+				(font
+					(size 1.27 1.27)
+				)
+				(hide yes)
+			)
+		)
+		(pin "1"
+		)
+		(pin "2"
+		)
+		(instances
+			(project ""
+				(path "/6275a1a7-d424-4390-b849-2e49b1a9780b"
+					(reference "LS1")
+					(unit 1)
+				)
+			)
+		)
+	)
+	(symbol
 		(lib_id "Device:R")
 		(at 110.49 39.37 0)
@@
 		(on_board yes)
 		(dnp no)
-		(fields_autoplaced yes)
 		(property "Reference" "Speaker1"
-			(at 82.55 54.6099 90)
+			(at 82.042 50.292 90)
 			(effects
 				(font
@@
 		)
 		(property "Value" "2_through_holes"
-			(at 82.55 57.1499 90)
+			(at 82.55 63.5 90)
 			(effects
 				(font

Commit message: changed rotations of components
Parts:
- USB-C1: footprint Connector_USB:USB_C_Receptacle_GCT_USB4110 -> Connector_USB:USB_C_Receptacle_GCT_USB4105-xx-A_16P_TopMnt_Horizontal
Changed lines of the file:
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@@
 			"AAAAAAAAAAAAAAAAAAAAAAAAAAAAAAAAAAAAAAAAAAAAAAAAAAAAAAAAAAAAAAAAAAAAAAAAAAAA"
 			"AAAAAAAAAAAAAAAAAAAAAAAAAAAAAAAAAAAAAAAAAAAAAAAAAAAAAAAAAAAAAAAAAAAAAAAAAAAA"
-			"AAAAAAAAAAAAAAAAAAAAAAAAAAAAAAAAAA=="
+			"AAAAAAAAAAAAAAAAAAAAAAAAAAAAAAAAAND/rMXQ/6zF0P+sxdD/rMXQ/6zF0P+sxdD/rMXQ/6zF"
+			"0P+sxdD/rMXQ/6zF0P+sxdD/rMXQ/6zF0P+sxdD/rMXQ/6zF0P+sxdD/rMXQ/5GR1P9bKdv/Wynb"
+			"/1sp2/9bKdv/Wynb/1sp2/9bKdv/Wynb/1sp2/9bKdv/Wynb/1sp2/9bKdv/Wynb/1sp2/9bKdv/"
+			"Wynb/1sp2/9bKdv/Wynb/1sp2/9bKdv/Wynb/1sp2/9bKdv/Wynb/1sp2/9bKdv/Wynb/1sp2/9b"
+			"Kdv/dl3X/6zF0P+sxdD/rMXQ/6zF0P+sxdD/rMXQ/6zF0P+sxdD/rMXQ/6zF0P+sxdD/rMXQ/6zF"
+			"0P+sxdD/rMXQ/6zF0P+sxdD/rMXQ/6zF0P+sxdD/rMXQ/6zF0P+sxdD/rMXQ/6zF0P+sxdD/rMXQ"
+			"/6zF0P+sxdD/rMXQ/6zF0P+sxdD/rMXQ/6zF0P+sxdD/rMXQ/6zF0P+sxdD/rMXQ/6zF0P+sxdD/"
+			"rMXQ/6zF0P+sxdD/rMXQ/6zF0P+sxdD/rMXQ/6zF0P+sxdD/rMXQ/6zF0P+sxdD/rMXQ/6zF0P+s"
+			"xdD/rMXQ/6zF0P+sxdD/rMXQ/6zF0P+sxdD/rMXQ/6zF0P+sxdD/rMXQ/6zF0P+sxdD/rMXQ/6zF"
+			"0P+sxdD/rMXQ/6zF0P+sxdD/rMXQ/6zF0P+sxdD/rMXQ/6zF0P+sxdD/rMXQ/6zF0P+sxdD/rMXQ"
+			"/6zF0P+sxdD/rMXQ/6zF0P+sxdD/rMXQ/6zF0P+sxdD/rMXQ/6zF0P+sxdD/q8TPoqK50AsAAAAA"
+			"AAAAAAAAAAAAAAAAAAAAAAAAAAAAAAAAAAAAAAAAAAAAAAAAAAAAAAAAAAAAAAAAAAAAAAAAAAAA"
+			"AAAAAAAAAAAAAAAAAAAAAAAAAAAAAAAAAAAAAAAAAAAAAAAAAAAAAAAAAAAAAAAAAAAAAAAAAAAA"
+			"AAAAAAAAAAAAAAAAAAAAAAAAAAAAAAAAAAAAAAAAAAAAAAAAAAAAAAAAAAAAAAAAAACqxtQSrMXQ"
+			"mqzF0P+sxdD/rMXQ/6zF0P+sxdD/rMXQ/6zF0P+sxdD/rMXQ/6zF0P+sxdD/rMXQ/6zF0P+sxdD/"
+			"rMXQ/6zF0P+sxdD/rMXQ/6zF0P+sxdD/rMXQ/6zF0P+sxdD/rMXQ/6zF0P+sxdD/rMXQ/6zF0P+s"
+			"xdD/rMXQ/6zF0P+sxdD/rMXQ/6zF0P+sxdD/rMXQ/6zF0P+sxdD/rMXQ/6zF0P+sxdD/rMXQ/6zF"
+			"0P+sxdD/rMXQ/6zF0P+sxdD/rMXQ/6zF0P+sxdD/rMXQ/6zF0P+sxdD/rMXQ/6zF0P+sxdD/rMXQ"
+			"/6zF0P+sxdD/rMXQ/6zF0P+sxdD/rMXQ/w=="
 		)
 	)
@@
 			"AAAAAAAAAAAAAAAAAAAAAAAAAAAAAAAAAAAAAAAAAAAAAAAAAAAAAAAAAAAAAAAAAAAAAAAAAAAA"
 			"AAAAAAAAAAAAAAAAAAAAAAAAAAAAAAAAAAAAAAAAAAAAAAAAAAAAAAAAAAAAAAAAAAAAAAAAAAAA"
-			"AAAAAAAAAAAAAAAAAA=="
+			"AAAAAAAAAAAAAAAAAADgOfzskQEAAOA5/OyRAQAA4Dn87JEBAADgOfzskQEAAOA5/OyRAQAA4Dn8"
+			"7JEBAADgOfzskQEAAOA5/OyRAQAA4Dn87JEBAADgOfzskQEAAOA5/OyRAQAA4Dn87JEBAADgOfzs"
+			"kQEAAOA5/OyRAQAA4Dn87JEBAADgOfzskQEAAOA5/OyRAQAA4Dn87JEBAADgOfzskQEAAOA5/OyR"
+			"AQAA4Dn87JEBAADgOfzskQEAAOA5/OyRAQAA4Dn87JEBAADgOfzskQEAAOA5/OyRAQAA4Dn87JEB"
+			"AADgOfzskQEAAOA5/OyRAQAA4Dn87JEBAADgOfzskQEAAOA5/OyRAQAA4Dn87JEBAADgOfzskQEA"
+			"AOA5/OyRAQAA4Dn87JEBAADgOfzskQEAAOA5/OyRAQAA4Dn87JEBAADgOfzskQEAAOA5/OyRAQAA"
+			"4Dn87JEBAADgOfzskQEAAOA5/OyRAQAA4Dn87JEBAADgOfzskQEAAOA5/OyRAQAA4Dn87JEBAADg"
+			"OfzskQEAAOA5/OyRAQAA4Dn87JEBAADgOfzskQEAAOA5/OyRAQAA4Dn87JEBAADgOfzskQEAAOA5"
+			"/OyRAQAA4Dn87JEBAADgOfzskQEAAOA5/OyRAQAA4Dn87JEBAADgOfzskQEAAOA5/OyRAQAA4Dn8"
+			"7JEBAADgOfzskQEAAOA5/OyRAQAA4Dn87JEBAADgOfzskQEAAOA5/OyRAQAA4Dn87JEBAADgOfzs"
+			"kQEAAOA5/OyRAQAA4Dn87JEBAADgOfzskQEAAOA5/OyRAQAA4Dn87JEBAADgOfzskQEAAOA5/OyR"
+			"AQAA4Dn87JEBAADgOfzskQEAAOA5/OyRAQAA4Dn87JEBAADgOfzskQEAAOA5/OyRAQAA4Dn87JEB"
+			"AADgOfzskQEAAOA5/OyRAQAA4Dn87JEBAADgOfzskQEAAOA5/OyRAQAA4Dn87JEBAADgOfzskQEA"
+			"AOA5/OyRAQAA4Dn87JEBAADgOfzskQEAAOA5/OyRAQAA4Dn87JEBAADgOfzskQEAAOA5/OyRAQAA"
+			"4Dn87JEBAADgOfzskQEAAOA5/OyRAQAA4Dn87JEBAADgOfzskQEAAOA5/OyRAQAA4Dn87JEBAADg"
+			"OfzskQEAAOA5/OyRAQAA4Dn87JEBAADgOfzskQEAAOA5/OyRAQAA4Dn87JEBAADgOfzskQEAAOA5"
+			"/OyRAQAA4Dn87JEBAADgOfzskQEAAOA5/OyRAQAA4Dn87JEBAADgOfzskQEAAOA5/OyRAQAA4Dn8"
+			"7JEBAADgOfzskQEAAOA5/OyRAQAA4Dn87JEBAADgOfzskQEAAOA5/OyRAQAA4Dn87JEBAADgOfzs"
+			"kQEAAOA5/OyRAQAA4A=="
 		)
 	)
@@
 			)
 		)
-		(property "Footprint" "Connector_USB:USB_C_Receptacle_GCT_USB4110"
+		(property "Footprint" "Connector_USB:USB_C_Receptacle_GCT_USB4105-xx-A_16P_TopMnt_Horizontal"
 			(at 260.35 135.89 0)
 			(effects
