File: whole_reader/reader/reader.kicad_sch (KiCad schematic)
At the start: 68 parts, among them U1 LM386M-1, U2 STM32F103C8T6, U3 MCP16301Hx-xCH, U4 TP3232N-SR, Y1 16MHz

Commit message: drobné úpravy schémy
Changed lines of the file:
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@@
 			"xdD/rMXQ/6zF0P+sxdD/rMXQ/6zF0P+sxdD/rMXQ/6zF0P+sxdD/rMXQ/6zF0P+sxdD/rMXQ/6zF"
 			"0P+sxdD/rMXQ/6zF0P+sxdD/rMXQ/6zF0P+sxdD/rMXQ/6zF0P+sxdD/rMXQ/6zF0P+sxdD/rMXQ"
-			"/6zF0P+sxdD/rMXQ/6zF0P+sxdD/rMXQ/w=="
+			"/6zF0P+sxdD/rMXQ/6zF0P+sxdD/rMXQ/wAAAAAAAAAAAAAAAAAAAAAAAAAAAAAAAAAAAAAAAAAA"
+			"AAAAAAAAAAAAAAAAAAAAAAAAAAAAAAAAAAAAAAAAAAAAAAAAAAAAAAAAAAAAAAAAAAAAAAAAAAAA"
+			"AAAAAAAAAAAAAAAAAAAAAAAAAAAAAAAAAAAAAAAAAAAAAAAAAAAAAAAAAAAAAAAAAAAAAAAAAAAA"
+			"AAAAAAAAAAAAAAAAAAAAAAAAAAAAAAAAAAAAAAAAAAAAAAAAAAAAAAAAAAAAAAAAAAAAAAAAAAAA"
+			"AAAAAAAAAAAAAAAAAAAAAAAAAAAAAAAAAAAAAAAAAAAAAAAAAAAAAAAAAAAAAAAAAAAAAAAAAAAA"
+			"AAAAAAAAAAAAAAAAAAAAAAAAAAAAAAAAAAAAAAAAAAAAAAAAAAAAAAAAAAAAAAAAAAAAAAAAAAAA"
+			"AAAAAAAAAAAAAAAAAAAAAAAAAAAAAAAAAAAAAAAAAAAAAAAAAAAAAAAAAAAAAAAAAAAAAAAAAAAA"
+			"AAAAAAAAAAAAAAAAAAAAAAAAAAAAAAAAAAAAAAAAAAAAAAAAAAAAAAAAAAAAAAAAAAAAAAAAAAAA"
+			"AAAAAAAAAAAAAAAAAAAAAAAAAAAAAAAAAAAAAAAAAAAAAAAAAAAAAAAAAAAAAAAAAAAAAAAAAAAA"
+			"AAAAAAAAAAAAAAAAAAAAAAAAAAAAAAAAAAAAAAAAAAAAAAAAAAAAAAAAAAAAAAAAAAAAAAAAAAAA"
+			"AAAAAAAAAAAAAAAAAAAAAAAAAAAAAAAAAAAAAAAAAAAAAAAAAAAAAAAAAAAAAAAAAAAAAAAAAAAA"
+			"AAAAAAAAAAAAAAAAAAAAAAAAAAAAAAAAAAAAAAAAAAAAAAAAAAAAAAAAAAAAAAAAAAAAAAAAAAAA"
+			"AAAAAAAAAAAAAAAAAAAAAAAAAAAAAAAAAAAAAAAAAAAAAAAAAAAAAAAAAAAAAAAAAAAAAAAAAAAA"
+			"AAAAAAAAAAAAAAAAAAAAAAAAAAAAAAAAAAAAAAAAAAAAAAAAAAAAAAAAAAAAAAAAAAAAAAAAAAAA"
+			"AAAAAAAAAAAAAAAAAAAAAAAAAAAAAAAAAAAAAAAAAAAAAAAAAAAAAAAAAAAAAAAAAAAAAAAAAAAA"
+			"AAAAAAAAAAAAAAAAAAAAAAAAAAAAAAAAAAAAAAAAAAAAAAAAAAAAAAAAAAAAAAAAAAAAAAAAAAAA"
+			"AAAAAAAAAAAAAAAAAAAAAAAAAAAAAAAAAAAAAAAAAAAAAAAAAAAAAAAAAAAAAAAAAAAAAAAAAAAA"
+			"AAAAAAAAAAAAAAAAAAAAAAAAAAAAAAAAAAAAAAAAAAAAAAAAAAAAAAAAAAAAAAAAAAAAAAAAAAAA"
+			"AAAAAAAAAAAAAAAAAAAAAAAAAAAAAAAAAMqD/H8AAHD4yoP8fwAAUPbKg/x/AAAA9sqD/H8AAFD1"
+			"yoP8fwAAoPbKg/x/AACg9cqD/H8AAFDHy4P8fwAAAADKg/x/AADwlMqD/H8AAPBzy4P8fwAAsPfK"
+			"g/x/AABw98qD/H8AADD3yoP8fwAA8PbKg/x/AADg9MqD/H8AADD4yoP8fwAA8PfKg/x/AADgQsuD"
+			"/H8AAPBEy4P8fwAAkELLg/x/AACgRMuD/H8AALD0yoP8fwAAwPPKg/x/AABg+cqD/H8AACD1yoP8"
+			"fwAA4ATKg/x/AABgBcqD/H8AAJAEyoP8fwAAEAXKg/x/AACARcuD/H8AACBGy4P8fwAAMEXLg/x/"
+			"AADQRcuD/H8AANAKy4P8fwAAkGHKg/x/AABQYcqD/H8AALBfyoP8fwAA8F/Kg/x/AAAwYMqD/H8A"
+			"AABhyoP8fwAAsGDKg/x/AADQYcqD/H8AAHBfyoP8fwAAMF/Kg/x/AABgYsqD/H8AACBiyoP8fwAA"
+			"4JnKg/x/AAAwmsqD/H8AAHBgyoP8fwAA8PvKg/x/AACArcqD/H8AAMCtyoP8fwAAMK7Kg/x/AACg"
+			"r8qD/H8AAOCvyoP8fwAAILDKg/x/AAAgasqD/H8AAABnyoP8fwAAUGfKg/x/AACwCMuD/H8AAAAJ"
+			"y4P8fwAAUAnLg/x/AACgCcuD/H8AAMDGyYP8fwAA8CXKg/x/AABgjsuD/H8AAKCOy4P8fwAAoJDL"
+			"g/x/AADwkMuD/H8AAFCTy4P8fwAAsJPLg/x/AAAw6MqD/H8AAIDoyoP8fwAAwOPJg/x/AAAQ5MmD"
+			"/H8AALDoyYP8fwAAEOnJg/x/AABgSMuD/H8AAJBIy4P8fwAAYErLg/x/AACgSsuD/H8AAKBMy4P8"
+			"fwAA8EzLg/x/AABQT8uD/H8AALBPy4P8fwAAYL3Kg/x/AACgvcqD/H8AAGDAyoP8fwAAsMDKg/x/"
+			"AADAw8qD/H8AACDEyoP8fwAAYMfKg/x/AADAx8qD/H8AAGAtyoP8fwAAkC3Kg/x/AADQOcuD/H8A"
+			"ACA6y4P8fwAAYJ7Lg/x/AACgnsuD/H8AAICgy4P8fwAA0KDLg/x/AADgosuD/H8AAECjy4P8fwAA"
+			"gKfLg/x/AADgp8uD/H8AAAC9y4P8fwAAAL7Lg/x/AAAAv8uD/H8AAADAy4P8fwAA4MLJg/x/AABg"
+			"EcqD/H8AACCeyoP8fwAAYF3Kg/x/AAAg4MmD/H8AACAjy4P8fwAAMK/Kg/x/AADwrsqD/H8AACCx"
+			"yoP8fwAA4LDKg/x/AAAArsqD/H8AAICyyoP8fwAAILLKg/x/AABAs8qD/H8AAOCyyoP8fwAAALTK"
+			"g/x/AACgs8qD/H8AANCsyoP8fwAAYLHKgw=="
 		)
 	)
@@
 			"/OyRAQAA4Dn87JEBAADgOfzskQEAAOA5/OyRAQAA4Dn87JEBAADgOfzskQEAAOA5/OyRAQAA4Dn8"
 			"7JEBAADgOfzskQEAAOA5/OyRAQAA4Dn87JEBAADgOfzskQEAAOA5/OyRAQAA4Dn87JEBAADgOfzs"
-			"kQEAAOA5/OyRAQAA4A=="
+			"kQEAAOA5/OyRAQAA4GJlWjFqcm9TUG9YK3NkSmRLT1ZQcE1LNXdQQWNyS1ZCUWNFODBvNWdSUVM0"
+			"NFhvTmlJNVUrTldWenBJM25tWlZETFhqSWxPMTh0cFFBOUhhV3lUd2UxRUx1cTRyWkJvK2NrM1Rk"
+			"WE9OVlhMQ2FuRUFLeXI1WHlvN2d2OVJWM3VDUTdJQmxoT29wSjBRSTR5MUhwUkhlWFQ0RjUrV3Vm"
+			"L3BuQksxREFrYWNYMmRsYVZ0ZXA1enR5ODNwN1BaRTZpbFE1S2pmTUJNQ3Z5NW5waGtuUkFvc2R1"
+			"ZC9HWjN5U1FFTkZEbHR5K0VLT1AyNk1OcmNpZEY4d1ZkK0FrYzAwRGRKSGVRMU82SkpDdTFBMXVI"
+			"ZWZvNC9ZWVF5dEt3eVNMNVYrY2xOenV6Vi8wY0pBQXVQQXlxRDNSbDBlQ0E3SWVsanNnTXd5MVNr"
+			"UnFzWWVoWEQ5RHJmWFFaZnh6N1gvK3dCazAxeWNqeHliYXJhdXM0ajR6clEzUW43bDM3WDkreTht"
+			"MDFLY1RpTVVzRTdxY1g4ekVrblJBdnVhM2lIYzJDT1VJeXdGZEl0L3A5bGp5OE1oeDZudklscWFX"
+			"NU1iYjJDZFN1U0U5NTBEV1J3djBaZDJMM1JpRTQ2U2xEbkE3YnFPZkJ1b3Nsc2x4U3VaTGZqUlVx"
+			"OG1OaG1vNUlEc1hFU01TbDFtOFpLNjVBYkp4NUJOM3l5TUhwUnFSenc1SWNqc2crMVBaVEd0eWlZ"
+			"ZkY0L0lJMDVqRnVUVFRSMk9WVGJKelFGN1huMHIvVUdSdVl5SGZjUW90OUttME9SOXJzUXZDU25D"
+			"Q3BBVzhHL2xtdStDOVFDcVJ6U0l2eVB6Qko2YW1iRUNNT1BVS1B2WkFkSm1ESUt6RzlEVFhORVJI"
+			"YXplMm95L3pmVnRTQm41MEcyYWozekV0NHEwYkdaZEhMZ0V0d0tSeTJWK2NKVHVhNnBXSTFPRkZ3"
+			"eHlzZjNLWDZ3b2d3S0dSajgxL3FtV3BtT2FBdERrZzljMlVGcGpua1NxZTZCRjRoWG5FWlRWdVhj"
+			"R2hOTlgrOFhKT3lVYUdOVmFkSHREU3Vld1ZhNmZIUFhZT1NGMHpwVndZR3ZuT1kwSVFWcDV6Wk9R"
+			"NDZwSHVqdkt1SmZxNDllTTREM0tnZWFVMGQ2QnFpTTdTbmpUZy9NaUhyNVBtZmVjdFpHUGNQbWVx"
+			"Vm9uSHhXNXB0MFJFR0VnVGM5bjVQR1N1V1pqb1N5UDJlZmJLU05vY2tIcG1Ta21lQUxFTXdMS1Ar"
+			"bDBQbldqd2l0L1ZMRkhkZk1xUStqY0srbldLblErd0RCUk0xZ0dKL25jTFFWajVUcHBmaU5FbmNu"
+			"NkNzTjQwVFZTeGhxbwAAAAAAAAAAAAAAAAAAAAAAAAAAAAAAAAAAAAAAAAAAAAAAAAAAAAAAAAAA"
+			"AAAAAAAAAAAAAAAAAAAAAAAAAAAAAAAAAAAAAAAAAAAAAAAAAAAAAAAAAAAAAAAAAAAAAAAAAAAA"
+			"AAAAAAAAAAAAAAAAAAAAAAAAAAAAAAAAAAAAAAAAAAAAAAAAAAAAAAAAAAAAAAAAAAAAAAAAAAAA"
+			"AAAAAAAAAAAAAAAAAAAAAAAAAAAAAAAAAAAAAAAAAAAAAAAAAAAAAAAAAAAAAAAAAAAAAAAAAAAA"
+			"AAAAAAAAAAAAAAAAAAAAAAAAAAAAAAAAAAAAAAAAAAAAAAAAAAAAAAAAAAAAAAAAAAAAAAAAAAAA"
+			"AAAAAAAAAAAAAAAAAAAAAAAAAAAAAAAAAAAAAAAAAAAAAAAAAAAAAAAAAAAAAAAAAAAAAAAAAAAA"
+			"AAAAAAAAAAAAAAAAAAAAAAAAAAAAAAAAAAAAAAAAAAAAAAAAAAAAAAAAAAAAAAAAAAAAAAAAAAAA"
+			"AAAA4Dn87JEBAADgOfzskQEAAOA5/OyRAQAA4Dn87JEBAADgOfzskQEAAOA5/OyRAQAA4Dn87JEB"
+			"AADgOfzskQEAAOA5/OyRAQAA4Dn87JEBAADgOfzskQEAAOA5/OyRAQAA4Dn87JEBAADgOfzskQEA"
+			"AOA5/OyRAQAA4Dn87JEBAADgOfzskQEAAOA5/OyRAQAA4Dn87JEBAADgOfzskQEAAOA5/OyRAQAA"
+			"4Dn87JEBAADgOfzskQEAAOA5/OyRAQAA4Dn87JEBAADgOfzskQEAAOA5/OyRAQAA4Dn87JEBAADg"
+			"OfzskQEAAOA5/OyRAQAA4Dn87JEBAADgOfzskQEAAOA5/OyRAQAA4Dn87JEBAADgOfzskQEAAOA5"
+			"/OyRAQAA4Dn87JEBAADgOfzskQEAAOA5/OyRAQAA4Dn87JEBAADgOfzskQEAAOA5/OyRAQAA4Dn8"
+			"7JEBAADgOfzskQEAAOA5/OyRAQAA4Dn87JEBAADgOfzskQEAAOA5/OyRAQAA4Dn87JEBAADgOfzs"
+			"kQEAAOA5/OyRAQAA4Dn87JEBAADgOfzskQEAAOA5/OyRAQAA4Dn87JEBAADgOfzskQEAAOA5/OyR"
+			"AQAA4Dn87JEBAADgOfzskQEAAOA5/OyRAQAA4Dn87JEBAADgOfzskQEAAOA5/OyRAQAA4Dn87JEB"
+			"AADgOfzskQEAAOA5/OyRAQAA4Dn87JEBAADgOfzskQEAAOA5/OyRAQAA4Dn87JEBAADgOfzskQEA"
+			"AOA5/OyRAQAA4Dn87JEBAADgOfzskQEAAOA5/OyRAQAA4Dn87JEBAADgOfzskQEAAOBiZVoxanJv"
+			"U1BvWCtzZEpkS09WUA=="
 		)
 	)
@@
 	)
 	(symbol
+		(lib_id "power:GND")
+		(at 72.39 185.42 0)
+		(unit 1)
+		(exclude_from_sim no)
+		(in_bom yes)
+		(on_board yes)
+		(dnp no)
+		(fields_autoplaced yes)
+		(property "Reference" "#PWR042"
+			(at 72.39 191.77 0)
+			(effects
+				(font
+					(size 1.27 1.27)
+				)
+				(hide yes)
+			)
+		)
+		(property "Value" "GND"
+			(at 72.39 190.5 0)
+			(effects
+				(font
+					(size 1.27 1.27)
+				)
+			)
+		)
+		(property "Footprint" ""
+			(at 72.39 185.42 0)
+			(effects
+				(font
+					(size 1.27 1.27)
+				)
+				(hide yes)
+			)
+		)
+		(property "Datasheet" ""
+			(at 72.39 185.42 0)
+			(effects
+				(font
+					(size 1.27 1.27)
+				)
+				(hide yes)
+			)
+		)
+		(property "Description" "Power symbol creates a global label with name \"GND\" , ground"
+			(at 72.39 185.42 0)
+			(effects
+				(font
+					(size 1.27 1.27)
+				)
+				(hide yes)
+			)
+		)
+		(pin "1"
+		)
+		(instances
+			(project "reader"
+				(path "/6275a1a7-d424-4390-b849-2e49b1a9780b"
+					(reference "#PWR042")
+					(unit 1)
+				)
+			)
+		)
+	)
+	(symbol
 		(lib_id "Amplifier_Audio:LM386")
 		(at 57.15 46.99 0)
@@
 		(dnp no)
 		(property "Reference" "C23"
-			(at 238.506 92.964 0)
+			(at 238.252 92.71 0)
 			(effects
 				(font
@@
 		)
 		(property "Value" "10 µF"
-			(at 237.49 98.044 0)
+			(at 236.22 98.044 0)
 			(effects
 				(font
@@
 	)
 	(symbol
-		(lib_id "power:GND")
-		(at 72.39 185.42 0)
-		(unit 1)
-		(exclude_from_sim no)
-		(in_bom yes)
-		(on_board yes)
-		(dnp no)
-		(fields_autoplaced yes)
-		(property "Reference" "#PWR09"
-			(at 72.39 191.77 0)
-			(effects
-				(font
-					(size 1.27 1.27)
-				)
-				(hide yes)
-			)
-		)
-		(property "Value" "GND"
-			(at 72.39 190.5 0)
-			(effects
-				(font
-					(size 1.27 1.27)
-				)
-				(hide yes)
-			)
-		)
-		(property "Footprint" ""
-			(at 72.39 185.42 0)
-			(effects
-				(font
-					(size 1.27 1.27)
-				)
-				(hide yes)
-			)
-		)
-		(property "Datasheet" ""
-			(at 72.39 185.42 0)
-			(effects
-				(font
-					(size 1.27 1.27)
-				)
-				(hide yes)
-			)
-		)
-		(property "Description" "Power symbol creates a global label with name \"GND\" , ground"
-			(at 72.39 185.42 0)
-			(effects
-				(font
-					(size 1.27 1.27)
-				)
-				(hide yes)
-			)
-		)
-		(pin "1"
-		)
-		(instances
-			(project "reader"
-				(path "/6275a1a7-d424-4390-b849-2e49b1a9780b"
-					(reference "#PWR09")
-					(unit 1)
-				)
-			)
-		)
-	)
-	(symbol
 		(lib_id "Device:R")
 		(at 41.91 31.75 0)
@@
 		(dnp no)
 		(property "Reference" "R1"
-			(at 39.624 34.798 90)
+			(at 36.576 31.75 90)
 			(effects
 				(font
 					(size 1.27 1.27)
 				)
-				(justify left)
 			)
 		)
 		(property "Value" "100 K"
-			(at 44.196 34.544 90)
+			(at 39.116 31.75 90)
 			(effects
 				(font
 					(size 1.27 1.27)
 				)
-				(justify left)
 			)
 		)
@@
 		(dnp no)
 		(property "Reference" "R2"
-			(at 37.084 43.18 90)
+			(at 36.576 44.45 90)
 			(effects
 				(font
 					(size 1.27 1.27)
 				)
-				(justify right)
 			)
 		)
 		(property "Value" "10 K"
-			(at 39.37 42.164 90)
+			(at 39.116 44.45 90)
 			(effects
 				(font
 					(size 1.27 1.27)
 				)
-				(justify right)
 			)
 		)

Commit message: added new conector for sp and low pass filter
Parts:
- removed LS1: Speaker, symbol Device:Speaker
- removed Speaker1: 2_through_holes, Connector_Wire:SolderWire-0.1sqmm_1x02_P3.6mm_D0.4mm_OD1mm, symbol Connector:Conn_01x01_Socket
- added C24: 470 nF, Capacitor_SMD:C_0603_1608Metric, symbol Device:C
- added Speaker1: 8 Ohm, Connector_Molex:Molex_PicoBlade_53047-0210_1x02_P1.25mm_Vertical, symbol UACS:Speaker
- C12, C15, C17, C2, C23: JLCPCB https://jlcpcb.com/partdetail/20411-CL10A106KP8NNNC/C19702 -> https://jlcpcb.com/partdetail/97651-CL10A106MA8NRNC/C96446; LCSC C19702 -> C96446
Connections:
- net GND: now also C24.2, Speaker1.2
- net at R1.2, R2.1: now also C24.1
- net at C9.2: now also Speaker1.1
Other:
- note added: "Low pass filter for 5-7 kHz"
- note added: "MAX V+: 12V MIN V+: 5V"
