File: V2/kicad/reader.kicad_pcb (KiCad board)
At the start: 2 copper layers, 42.5 x 62 mm, 93 parts, among them SW1 SW_Rezistance, SW2 SW_src, U1 STM32H523CET6, U2 MAX98357AETE+T, U3 MLD-TF PUSH-H18, U4 TCAN1057AVDRQ1, U5 ESD2CAN24-ES, U6 RJ-064-1, U7 MCP16301Hx-xCH, Y1 16MHz

Commit message: updated pdf with better images of pcb
Routing:
- net GND: vias 186 -> 187
Changed lines of the file:
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@@
 		(grid_origin 133 28)
 		(pcbplotparams
-			(layerselection 0x00000000_00000000_55555555_55555551)
-			(plot_on_all_layers_selection 0x00000000_00000000_00000000_02002022)
+			(layerselection 0x00000000_00000000_55555555_55555554)
+			(plot_on_all_layers_selection 0x00000000_00000000_00000000_02000000)
 			(disableapertmacros no)
 			(usegerberextensions no)
@@
 			(dashed_line_dash_ratio 12)
 			(dashed_line_gap_ratio 3)
-			(svgprecision 4)
+			(svgprecision 6)
 			(plotframeref no)
 			(mode 1)
@@
 			(psnegative no)
 			(psa4output no)
-			(plot_black_and_white yes)
+			(plot_black_and_white no)
 			(sketchpadsonfab no)
 			(plotpadnumbers no)
@@
 			(crossoutdnponfab yes)
 			(subtractmaskfromsilk no)
-			(outputformat 1)
+			(outputformat 5)
 			(mirror no)
-			(drillshape 0)
+			(drillshape 2)
 			(scaleselection 1)
 			(outputdirectory "")
@@
 				(font
 					(size 1.27 1.27)
+					(thickness 0.15)
 				)
 			)
@@
 		(size 0.6)
 		(drill 0.3)
+		(layers "F.Cu" "B.Cu")
+		(free yes)
+		(net "GND")
+	)
+	(via
+		(at 59.78 88.54)
+		(size 0.6)
+		(drill 0.3)
